File: Hardware/GSMLinkModem/GSMLinkModem.sch (KiCad schematic (older format))
At the start: 47 parts

Commit message: new: Work in progress
Parts:
- removed C? (x2): 0.1uF, Capacitor_SMD:C_0805_2012Metric_Pad1.18x1.45mm_HandSolder, symbol Device:C
- removed R?: 510R, Resistor_SMD:R_0805_2012Metric_Pad1.15x1.40mm_HandSolder, symbol Device:R
- added C? (x2): 0.1uF, Capacitor_SMD:C_0805_2012Metric_Pad1.18x1.45mm_HandSolder, symbol Device:C
- added C? (x6): 10uF, Capacitor_SMD:C_1206_3216Metric_Pad1.42x1.75mm_HandSolder, symbol Device:C
- added L?: 2.2uH, Inductor_SMD:L_1008_2520Metric_Pad1.43x2.20mm_HandSolder, symbol Device:L
- added R? (x2): 510R, Resistor_SMD:R_0805_2012Metric_Pad1.15x1.40mm_HandSolder, symbol Device:R
- added R? (x2): 10K, Resistor_SMD:R_0805_2012Metric_Pad1.15x1.40mm_HandSolder, symbol Device:R
- added U?: TPS63900, Package_DFN_QFN:DFN-10-1EP_3x3mm_P0.5mm_EP1.65x2.38mm_ThermalVias, symbol mylib-symbols:TPS63900
Connections:
- net labels added: FLASH_PWR, HOLD, SCK, SI, SO, V_SELECT, WP
- wire segments 138 -> 193
Other:
- note added: "Accelerometer LIS3DHTR 16-LGA (3x3)"
- note added: "FLASH - NOR 32Mb (4M x 8) SPI"
- note added: "Power swith control"
- moved on the sheet: C?, FB?, Q?, R?, SW?, U?, Y?

Commit message: new: Work in progress
Parts:
- removed C? (x2): 0.1uF, Capacitor_SMD:C_0805_2012Metric_Pad1.18x1.45mm_HandSolder, symbol Device:C
- removed C? (x3): 10uF, Capacitor_SMD:C_1206_3216Metric_Pad1.42x1.75mm_HandSolder, symbol Device:C
- removed Q?: BC847C, Package_TO_SOT_SMD:SOT-23, symbol Transistor_BJT:BC847
- removed Q?: AO3419, Package_TO_SOT_SMD:SOT-23, symbol Transistor_FET:AO3401A
- removed R? (x2): 10K, Resistor_SMD:R_0805_2012Metric_Pad1.15x1.40mm_HandSolder, symbol Device:R
- removed R?: 510R, Resistor_SMD:R_0805_2012Metric_Pad1.15x1.40mm_HandSolder, symbol Device:R
- removed U?: EFM32TG11B320F128GQ64-B, Package_QFP:TQFP-64_10x10mm_P0.5mm, symbol mylib-symbols:EFM32TG11B320F128GQ64-B
- removed U?: BC66, RF_GSM:Quectel_BC66, symbol RF_GSM:BC66
- removed U?: AT25SF321B-SSHB-T, Package_SO:SOIC-8_3.9x4.9mm_P1.27mm, symbol mylib-symbols:AT25SF321B-SSHB-T
- removed U?: TPS63900, Package_DFN_QFN:DFN-10-1EP_3x3mm_P0.5mm_EP1.65x2.38mm_ThermalVias, symbol mylib-symbols:TPS63900
- added C? (x2): 10nF, Capacitor_SMD:C_0805_2012Metric_Pad1.18x1.45mm_HandSolder, symbol Device:C
- added C? (x3): 10uF, Capacitor_SMD:C_1206_3216Metric_Pad1.42x1.75mm_HandSolder, symbol Device:C
- added C?: 1uF, Capacitor_SMD:C_0805_2012Metric_Pad1.18x1.45mm_HandSolder, symbol Device:C
- added C? (x3): 820uF, Capacitor_THT:CP_Radial_D8.0mm_P3.50mm, symbol Device:CP1
- added C? (x3): 0.1uF, Capacitor_SMD:C_0805_2012Metric_Pad1.18x1.45mm_HandSolder, symbol Device:C
- added D?: LED, symbol Device:LED
- added Q? (x4): BC847C, Package_TO_SOT_SMD:SOT-23, symbol Transistor_BJT:BC847
- added R? (x8): 10K, Resistor_SMD:R_0805_2012Metric_Pad1.15x1.40mm_HandSolder, symbol Device:R
- added R? (x3): 2K, Resistor_SMD:R_0805_2012Metric_Pad1.15x1.40mm_HandSolder, symbol Device:R
- added R? (x2): 5.9K, Resistor_SMD:R_0805_2012Metric_Pad1.15x1.40mm_HandSolder, symbol Device:R
- added R? (x6): 470R, Resistor_SMD:R_0805_2012Metric_Pad1.15x1.40mm_HandSolder, symbol Device:R
- added R?: 22R, Resistor_SMD:R_0805_2012Metric_Pad1.15x1.40mm_HandSolder, symbol Device:R
- added SW?: SW_DIP_x02, symbol Switch:SW_DIP_x02
- added TP? (x2): 3V3_line, TestPoint:TestPoint_THTPad_D1.5mm_Drill0.7mm, symbol Connector:TestPoint
- added TP?: DC/DC_line, TestPoint:TestPoint_THTPad_D1.5mm_Drill0.7mm, symbol Connector:TestPoint
- added TP?: VBAT_line, TestPoint:TestPoint_THTPad_D1.5mm_Drill0.7mm, symbol Connector:TestPoint
- added U?: MIC29302WU, Package_TO_SOT_SMD:TO-263-5_TabPin3, symbol Regulator_Linear:MIC29302WU
- added U?: BC66NADA-04-STD, RF_GSM:Quectel_BC66, symbol mylib-symbols:BC66NADA-04-STD
- added U?: TPS63900, Package_DFN_QFN:DFN-10-1EP_3x3mm_P0.5mm_EP1.65x2.38mm_ThermalVias, symbol mylib-symbols:TPS63900
- added U?: AT25SF321B-SSHB-T, Package_SO:SOIC-8_3.9x4.9mm_P1.27mm, symbol mylib-symbols:AT25SF321B-SSHB-T
- added U?: EFM32TG11B320F128GQ64-B, Package_QFP:TQFP-64_10x10mm_P0.5mm, symbol mylib-symbols:EFM32TG11B320F128GQ64-B
- added U?: ISL21080DIH310Z-TK, Package_TO_SOT_SMD:SOT-23_Handsoldering, symbol mylib-symbols:ISL21080DIH310Z-TK
- R? (x2): Description 10 kOhms ±5% 0.125W, 1/8W Chip Resistor 0805 (2012 Metric) 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 -> 10 kOhms ±1% 0.125W, 1/8W Chip Resistor 0805 (2012 Metric) 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; PartNumber RC0805JR-0710KL -> RC0805FR-0710KP
Connections:
- net labels added: +1V8, +BATT, 3V3_ENBL, BC66_NET_LED, BC66_PWR, BC66_PWRKEY, BC66_RESET, BC66_RST, BC66_RXD, BC66_RXD_AUX, BC66_RXD_DBG, BC66_SLEEP, BC66_TXD, BC66_TXD_AUX, BC66_TXD_DBG, SW_ENBL, VCC
- net labels removed: FLASH_PWR
- wire segments 193 -> 294
Other:
- note added: "BC66 network LED"
- note added: "BC66 power on/off"
- note added: "BC66 reset control"
- note added: "BC66 sleep control"
- note added: "Filter to reduce noise at AVDD pin (1x10uF+2x0.1uF) + 1.024V micropower referece"
- note added: "RESET button"
- note added: "VCC may be in range 3.6V-4V"
- note removed: "Low-pass filter for AVDD power rail\n"
- note removed: "Power swith control"
- moved on the sheet: C?, FB?, J?, L?, Q?, R?, SW?, U?, Y?

Commit message: new: Work in progress
Parts:
- removed D?: LED, symbol Device:LED
- removed Q? (x2): BC847C, Package_TO_SOT_SMD:SOT-23, symbol Transistor_BJT:BC847
- removed R?: 4.7K, Resistor_SMD:R_0805_2012Metric_Pad1.15x1.40mm_HandSolder, symbol Device:R
- removed R? (x2): 10K, Resistor_SMD:R_0805_2012Metric_Pad1.15x1.40mm_HandSolder, symbol Device:R
- removed R? (x2): 470R, Resistor_SMD:R_0805_2012Metric_Pad1.15x1.40mm_HandSolder, symbol Device:R
- removed R?: 2K, Resistor_SMD:R_0805_2012Metric_Pad1.15x1.40mm_HandSolder, symbol Device:R
- removed SW?: SW_DIP_x02, symbol Switch:SW_DIP_x02
- added C? (x3): 10uF, Capacitor_SMD:C_1206_3216Metric_Pad1.42x1.75mm_HandSolder, symbol Device:C
- added C? (x4): 10nF, Capacitor_SMD:C_0805_2012Metric_Pad1.18x1.45mm_HandSolder, symbol Device:C
- added C? (x6): 0.1uF, Capacitor_SMD:C_0805_2012Metric_Pad1.18x1.45mm_HandSolder, symbol Device:C
- added C? (x9): 18pF, Capacitor_SMD:C_0805_2012Metric_Pad1.18x1.45mm_HandSolder, symbol Device:C
- added C?: 1uF, Capacitor_SMD:C_0805_2012Metric_Pad1.18x1.45mm_HandSolder, symbol Device:C
- added C? (x2): DNP, Capacitor_SMD:C_0402_1005Metric_Pad0.74x0.62mm_HandSolder, symbol Device:C
- added D?: ESDA6V1-5SC6, Package_TO_SOT_SMD:SOT-23-6, symbol Power_Protection:ESDA6V1-5SC6
- added D?: SM6T7V5A, Diode_SMD:D_SMB, symbol Diode:SM6T7V5A
- added J? (x3): Conn_01x04_Male, symbol Connector:Conn_01x04_Male
- added J?: 1909763-1, digikey-footprints:UMCoax_Pin_1909763-1, symbol Connector:Conn_Coaxial
- added J?: Conn_01x02_Male, symbol Connector:Conn_01x02_Male
- added Q? (x2): AO3419, Package_TO_SOT_SMD:SOT-23, symbol Transistor_FET:AO3401A
- added Q? (x3): BC847C, Package_TO_SOT_SMD:SOT-23, symbol Transistor_BJT:BC847
- added R?: DNP, Resistor_SMD:R_0805_2012Metric_Pad1.15x1.40mm_HandSolder, symbol Device:R
- added R?: 0R, Resistor_SMD:R_0805_2012Metric_Pad1.15x1.40mm_HandSolder, symbol Device:R
- added R? (x4): 470R, Resistor_SMD:R_0805_2012Metric_Pad1.15x1.40mm_HandSolder, symbol Device:R
- added R? (x8): 10K, Resistor_SMD:R_0805_2012Metric_Pad1.15x1.40mm_HandSolder, symbol Device:R
- added R? (x18): 22R, Resistor_SMD:R_0805_2012Metric_Pad1.15x1.40mm_HandSolder, symbol Device:R
- added R?: 4.7K, Resistor_SMD:R_0805_2012Metric_Pad1.15x1.40mm_HandSolder, symbol Device:R
- added R?: 0R, Resistor_SMD:R_0402_1005Metric_Pad0.72x0.64mm_HandSolder, symbol Device:R
- added R?: 3M, Resistor_SMD:R_0805_2012Metric_Pad1.15x1.40mm_HandSolder, symbol Device:R
- added R?: 1M, Resistor_SMD:R_0805_2012Metric_Pad1.15x1.40mm_HandSolder, symbol Device:R
- added TP?: GND, TestPoint:TestPoint_THTPad_D1.5mm_Drill0.7mm, symbol Connector:TestPoint
- R?: value 22R -> 0R; Description 22 Ohms ±5% 0.125W, 1/8W Chip Resistor 0805 (2012 Metric) T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 -> 0 Ohms 0.125W, 1/8W Chip Resistor 0805 (2012 Metric) Thick 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; PartNumber RC0805JR-0722RL -> RC0805JR-070RL
- TP?: value DC/DC_line -> 4V_line
Connections:
- net labels added: +4V, BC66_ON_OFF, BC66_RI, EXT_RXD, EXT_RXD_DBG, EXT_TXD, EXT_TXD_DBG, FLASH_PWR, MCU_CLK, MCU_CS, MCU_EM4WU4, MCU_MISO, MCU_MOSI, MCU_RESET, MCU_RI, MCU_SWCLK, MCU_SWDIO, NET_STATUS, SIM_CLK, SIM_DATA, SIM_RST, SIM_VDD
- net labels removed: BC66_NET_LED, BC66_SLEEP, HOLD, MCU_RX2, MCU_RX3, MCU_TX2, MCU_TX3, SCK, SI, SO, VCC, WP
- wire segments 294 -> 514
Other:
- note added: "+V"
- note added: "3V3<->1V8 signal levels translator"
- note added: "BC66 PWR key"
- note added: "Connect reed switch here"
- note added: "FLASH SPI"
- note added: "FLASH power on/off"
- note added: "GND"
- note added: "I2C bus"
- note added: "MCU UART"
- note added: "Modem aux UART"
- note added: "Modem main UART"
- note added: "NB-IoT modem BC66-NA"
- note added: "Optional power jumpers"
- note added: "Pin to wake-up MCU from EM4 sleep"
- note added: "Power supply controller TPS63900 + MIC29302WU"
- note added: "Pulse"
- note added: "RX"
- note added: "SIG"
- note added: "SWD"
- note added: "TX"
- note added: "Test points"
- note added: "UART0"
- note added: "UART1 + modem control"
- note added: "Use 3V3 jumper for BC66-NA modem\n"
- note added: "Use 4V jumper for M66 modem"
- note added: "VBAT voltage monitor"
- note removed: "BC66 network LED"
- note removed: "BC66 sleep control"
- moved on the sheet: C?, FB?, J?, L?, Q?, R?, SW?, TP?, U?, Y?

Commit message: new: Work in progress
Parts:
- removed C?: 820uF, Capacitor_THT:CP_Radial_D8.0mm_P3.50mm, symbol Device:CP1
- removed C? (x4): 18pF, Capacitor_SMD:C_0805_2012Metric_Pad1.18x1.45mm_HandSolder, symbol Device:C
- removed C? (x2): 0.1uF, Capacitor_SMD:C_0805_2012Metric_Pad1.18x1.45mm_HandSolder, symbol Device:C
- removed R?: DNP, Resistor_SMD:R_0805_2012Metric_Pad1.15x1.40mm_HandSolder, symbol Device:R
- removed R?: 0R, Resistor_SMD:R_0805_2012Metric_Pad1.15x1.40mm_HandSolder, symbol Device:R
- removed R?: 10K, Resistor_SMD:R_0805_2012Metric_Pad1.15x1.40mm_HandSolder, symbol Device:R
- removed R?: 5.9K, Resistor_SMD:R_0805_2012Metric_Pad1.15x1.40mm_HandSolder, symbol Device:R
- removed R?: 470R, Resistor_SMD:R_0805_2012Metric_Pad1.15x1.40mm_HandSolder, symbol Device:R
- removed R? (x8): 22R, Resistor_SMD:R_0805_2012Metric_Pad1.15x1.40mm_HandSolder, symbol Device:R
- removed U?: MIC29302WU, Package_TO_SOT_SMD:TO-263-5_TabPin3, symbol Regulator_Linear:MIC29302WU
- added C10: 10uF, Capacitor_SMD:C_1206_3216Metric_Pad1.42x1.75mm_HandSolder, symbol Device:C
- added C2, C20, C3: 0.1uF, Capacitor_SMD:C_0805_2012Metric_Pad1.18x1.45mm_HandSolder, symbol Device:C
- added C23, C25, C27, C5, C6, C8, C9: 18pF, Capacitor_SMD:C_0805_2012Metric_Pad1.18x1.45mm_HandSolder, symbol Device:C
- added C4: 820uF, Capacitor_THT:CP_Radial_D8.0mm_P3.50mm, symbol Device:CP1
- added D1, D10, D11, D12, D14, D3, D4, D5, D6, D7, D8, D9: PESD5V0L1UA,115, Diode_SMD:D_SOD-323_HandSoldering, symbol Diode:SM6T7V5A
- added F1: 0ZCJ0100FF2E, Fuse:Fuse_1206_3216Metric_Pad1.42x1.75mm_HandSolder, symbol Device:Polyfuse
- added J1: Screw_Terminal_01x02, symbol Connector:Screw_Terminal_01x02
- added J4: Conn_01x05_Male, symbol Connector:Conn_01x05_Male
- added R17, R18, R19, R5, R6, R7, R8: 22R, Resistor_SMD:R_0805_2012Metric_Pad1.15x1.40mm_HandSolder, symbol Device:R
- added R26: 16.2K, Resistor_SMD:R_0805_2012Metric_Pad1.15x1.40mm_HandSolder, symbol Device:R
- added R28: 8.25K, Resistor_SMD:R_0805_2012Metric_Pad1.15x1.40mm_HandSolder, symbol Device:R
- added R32, R33: 5.11K, Resistor_SMD:R_0805_2012Metric_Pad1.15x1.40mm_HandSolder, symbol Device:R
- added U4: MIC5504-3.3YM5, Package_TO_SOT_SMD:SOT-23-5, symbol Regulator_Linear:MIC5504-3.3YM5
- D13: renamed from D?; value SM6T7V5A -> PESD5V0L1UA,115; footprint Diode_SMD:D_SMB -> Diode_SMD:D_SOD-323_HandSoldering; Description (none) -> 5V 3.5A (8/20µs) Ipp ESD protection TVS Diode Surface Mount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; PartNumber (none) -> PESD5V0L1UA,115
- TP3: renamed from TP?; value 4V_line -> VCC_line
- gave numbers to parts that had none: 133
Connections:
- net labels added: VBUS, VCC
- net labels removed: +4V
- wire segments 514 -> 590
Other:
- note added: "1x10uF bulk decoupling + 100nF per power pin"
- note added: "External connectors"
- note added: "MCU SWD"
- note added: "Modem debug UART"
- note added: "Power control"
- note added: "Power select\nPull V_SEL high for M66 modem (4V output)\nPull V_SEL low for BC66-NA modem (3.3V output)"
- note added: "SIM card slot"
- note added: "SWCLK"
- note added: "SWDIO"
- note added: "UART1 (modem control)"
- note added: "VBAT in"
- note added: "VCC: 3.3V or 4V"
- note added: "~RESET~"
- note removed: "1x 10uF bulk decoupling + 100nF per power pin"
- note removed: "Modem aux UART"
- note removed: "Optional power jumpers"
- note removed: "UART1 + modem control"
- note removed: "Use 3V3 jumper for BC66-NA modem\n"
- note removed: "Use 4V jumper for M66 modem"
- note removed: "VCC may be in range 3.6V-4V"
- moved on the sheet: C1, C11, C12, C13, C14, C15, C16, C17, C18, C19, C21, C22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

Commit message: new: Work in progress
Parts:
- removed C15: 820uF, Capacitor_THT:CP_Radial_D8.0mm_P3.50mm, symbol Device:CP1
- removed C19: 18pF, Capacitor_SMD:C_0805_2012Metric_Pad1.18x1.45mm_HandSolder, symbol Device:C
- removed C24: 0.1uF, Capacitor_SMD:C_0805_2012Metric_Pad1.18x1.45mm_HandSolder, symbol Device:C
- removed C28: 1uF, Capacitor_SMD:C_0805_2012Metric_Pad1.18x1.45mm_HandSolder, symbol Device:C
- removed C30: 10uF, Capacitor_SMD:C_1206_3216Metric_Pad1.42x1.75mm_HandSolder, symbol Device:C
- removed D14: PESD5V0L1UA,115, Diode_SMD:D_SOD-323_HandSoldering, symbol Diode:SM6T7V5A
- removed FB2: 1 kOhms @ 100MHz, Inductor_SMD:L_0805_2012Metric_Pad1.15x1.40mm_HandSolder, symbol Device:Ferrite_Bead
- removed J3: Conn_01x04_Male, symbol Connector:Conn_01x04_Male
- removed Q8: AO3419, Package_TO_SOT_SMD:SOT-23, symbol Transistor_FET:AO3401A
- removed Q9: BC847C, Package_TO_SOT_SMD:SOT-23, symbol Transistor_BJT:BC847
- removed R25: 10K, Resistor_SMD:R_0805_2012Metric_Pad1.15x1.40mm_HandSolder, symbol Device:R
- removed R33: 5.11K, Resistor_SMD:R_0805_2012Metric_Pad1.15x1.40mm_HandSolder, symbol Device:R
- removed R36: 4.7K, Resistor_SMD:R_0805_2012Metric_Pad1.15x1.40mm_HandSolder, symbol Device:R
- removed R37: 2K, Resistor_SMD:R_0805_2012Metric_Pad1.15x1.40mm_HandSolder, symbol Device:R
- removed R38: 510R, Resistor_SMD:R_0805_2012Metric_Pad1.15x1.40mm_HandSolder, symbol Device:R
- removed R39: 470R, Resistor_SMD:R_0805_2012Metric_Pad1.15x1.40mm_HandSolder, symbol Device:R
- removed R40: 22R, Resistor_SMD:R_0805_2012Metric_Pad1.15x1.40mm_HandSolder, symbol Device:R
- removed R42: 0R, Resistor_SMD:R_0805_2012Metric_Pad1.15x1.40mm_HandSolder, symbol Device:R
- removed TP5: 3V3_line, TestPoint:TestPoint_THTPad_D1.5mm_Drill0.7mm, symbol Connector:TestPoint
- removed U5: ISL21080DIH310Z-TK, Package_TO_SOT_SMD:SOT-23_Handsoldering, symbol mylib-symbols:ISL21080DIH310Z-TK
- added C25, C27: 10nF, Capacitor_SMD:C_0805_2012Metric_Pad1.18x1.45mm_HandSolder, symbol Device:C
- added D11, D13: PESD5V0L1UA,115, Diode_SMD:D_SOD-323_HandSoldering, symbol Diode:SM6T7V5A
- added D16: LED_RED, LED_SMD:LED_0805_2012Metric_Pad1.15x1.40mm_HandSolder, symbol Device:LED
- added D17: LED_GREEN, LED_SMD:LED_0805_2012Metric_Pad1.15x1.40mm_HandSolder, symbol Device:LED
- added J2: KLS1-207-1-04-S, Connector_PinHeader_2.54mm:PinHeader_1x04_P2.54mm_Vertical, symbol Connector:Conn_01x04_Male
- added J6: KLS2-308V-2.54-03P-4S, TerminalBlock_TE-Connectivity:TerminalBlock_TE_282834-3_1x03_P2.54mm_Horizontal, symbol Connector:Screw_Terminal_01x03
- added R16, R27: 10K, Resistor_SMD:R_0805_2012Metric_Pad1.15x1.40mm_HandSolder, symbol Device:R
- added R20, R22: 22R, Resistor_SMD:R_0805_2012Metric_Pad1.15x1.40mm_HandSolder, symbol Device:R
- added R21, R52, R53: 470R, Resistor_SMD:R_0805_2012Metric_Pad1.15x1.40mm_HandSolder, symbol Device:R
- added U4: ISL21080DIH310Z-TK, Package_TO_SOT_SMD:SOT-23_Handsoldering, symbol mylib-symbols:ISL21080DIH310Z-TK
- C22: value 10nF -> 0.1uF; Description 10000pF ±5% 100V Ceramic Capacitor C0G, NP0 1206 (3216 Metr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 -> 0.1µF ±10% 25V Ceramic Capacitor X7R 0805 (2012 Metric); PartNumber CC1206JKNPO0BN103 -> CC0805KRX7R8BB104; Voltage 100V -> 25V
- C42: renamed from C48; value 18pF -> DNP
- C47: renamed from C52; value 18pF -> DNP
- D1: renamed from D2; Description (none) -> Clamp 6.1V 100W TVS Diode Array Surface Mount SOT-23-6; PartNumber (none) -> ESDA6V1-5SC6
- J1: renamed from J2; value Conn_01x04_Male -> KLS1-207-1-04-S; footprint (none) -> Connector_PinHeader_2.54mm:PinHeader_1x04_P2.54mm_Vertical; Description (none) -> Connector Header Through Hole 4 position 0.100\" (2.54mm); PartNumber (none) -> KLS1-207-1-04-S
- J3: renamed from J4; value Conn_01x05_Male -> KLS1-207-1-05-S; footprint (none) -> Connector_PinHeader_2.54mm:PinHeader_1x05_P2.54mm_Vertical; Description (none) -> Connector Header Through Hole 5 position 0.100\" (2.54mm); PartNumber (none) -> KLS1-207-1-05-S
- J4: renamed from J1; value Screw_Terminal_01x02 -> KLS2-308V-2.54-02P-4S; footprint (none) -> TerminalBlock_TE-Connectivity:TerminalBlock_TE_282834-2_1x02_P2.54mm_Horizontal; Description (none) -> 2 Position Wire to Board Terminal Block Horizontal with Boa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; PartNumber (none) -> KLS2-308V-2.54-02P-4S
- J5: value SIM_Card_Shielded -> SIM8051-6-0-14-00-A; footprint (none) -> mylib-footprints:GCT_SIM8051-6-0-14-00-X-REVD; Description (none) -> 6 Position Card Connector NANO SIM Surface Mount, Right Ang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; PartNumber (none) -> SIM8051-6-0-14-00-A
- J7: value Conn_01x04_Male -> KLS1-207-1-04-S; footprint (none) -> Connector_PinHeader_2.54mm:PinHeader_1x04_P2.54mm_Vertical; Description (none) -> Connector Header Through Hole 4 position 0.100\" (2.54mm); PartNumber (none) -> KLS1-207-1-04-S
- J8: renamed from J6; value Conn_01x02_Male -> KLS1-207-1-02-S; footprint (none) -> Connector_PinHeader_2.54mm:PinHeader_1x02_P2.54mm_Vertical; Description (none) -> Connector Header Through Hole 2 position 0.100\" (2.54mm); PartNumber (none) -> KLS1-207-1-02-S
- R29: value 5.9K -> 10K; Description 5.9 kOhms ±1% 0.125W, 1/8W Chip Resistor 0805 (2012 Metric)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 -> 10 kOhms ±1% 0.125W, 1/8W Chip Resistor 0805 (2012 Metric) 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; PartNumber RC0805FR-075K9L -> RC0805FR-0710KP
- U1: footprint RF_GSM:Quectel_BC66 -> mylib-footprints:Quectel_BC66
- U2: renamed from U3; Description (none) -> Voltage Level Translator Bidirectional 1 Circuit 8 Channel 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; PartNumber (none) -> TXS0108EPW
- U6: renamed from U4; Description (none) -> Linear Voltage Regulator IC 1 Output 3.3V 300mA SOT-23-5; PartNumber (none) -> MIC5504-3.3YM5
- U8: Description (none) -> Accelerometer X, Y, Z Axis ±2g, 4g, 8g, 16g 0.5Hz ~ 625Hz 1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; PartNumber (none) -> LIS3DH
- U9: footprint Package_DFN_QFN:DFN-6-1EP_3x3mm_P1mm_EP1.65x2.55mm -> Package_DFN_QFN:DFN-6-1EP_3x3mm_P1mm_EP1.5x2.4mm
- Y2: value 48MHz -> DNP
- renumbered C2 to C1, C7 to C10, C25 to C11, C11 to C12, C12 to C13, C27 to C14, C13 to C15, C14 to C16, C21 to C19, C3 to C2, C4 to C20, C26 to C21, C10 to C23, C29 to C24, C32 to C26, C31 to C28, C16 to C29, C1 to C3, C34 to C30, C33 to C31, C35 to C32, C36 to C33, C37 to C34, C38 to C35, C40 to C36, C43 to C37, C45 to C38, C20 to C4, C46 to C40, C47 to C41, C41 to C43, C49 to C44, C50 to C45, C42 to C46, C44 to C48, C53 to C49, C54 to C50, C55 to C51, C56 to C52, C57 to C53, C51 to C54, C58 to C55, C59 to C56, C60 to C57, C61 to C58, C62 to C59, C63 to C60, C64 to C61, C65 to C62, C66 to C63, C8 to C7, C9 to C8, C23 to C9, D1 to D10, D11 to D12, D12 to D14, D13 to D15, D3 to D2, D4 to D3, D5 to D4, D6 to D5, D8 to D6, D9 to D7, D10 to D8, D7 to D9, J8 to J9, R5 to R1, R17 to R12, R18 to R13, R19 to R14, R12 to R15, R13 to R17, R14 to R18, R15 to R19, R6 to R2, R21 to R25, R22 to R26, R27 to R28, R7 to R3, R31 to R30, R30 to R31, R34 to R32, R16 to R33, R35 to R34, R20 to R35, R26 to R36, R41 to R37, R28 to R38, R32 to R39, R8 to R4, R44 to R40, R45 to R41, R46 to R42, R47 to R43, R48 to R44, R49 to R45, R50 to R46, R51 to R47, R52 to R48, R53 to R49, R1 to R5, R54 to R50, R43 to R51, R55 to R54, R56 to R55, R2 to R6, R3 to R7, R4 to R8, U2 to U3, U6 to U5
Connections:
- net +BATT: now also C22.1, R21.2
- net GND: now also C22.2, J4.2 (Pin_2), R29.2, C25.2, C27.2, D11.2 (A2), D13.2 (A2), D16.1 (K), D17.1 (K), J2.2 (Pin_2), R27.2, U4.3 (GND); no longer J4.1 (Pin_1)
- net MCU_EM4WU4: now also R29.1, C27.1, D13.1 (A1), R20.1; no longer C32.1, D15.1 (A1), R26.1, R31.1
- net SDO: now also U7.57 (PE8)
- net SIM_VDD: now also R16.2
- net VBUS: now also J4.1 (Pin_1), J2.4 (Pin_4); no longer J4.2 (Pin_2)
- net VDDA: now also U4.2 (VOUT)
- net at C15.1, D1.6 (IO5), J5.7 (I/O)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: now also R16.1
- net at C41.1, C45.1, FB1.2: now also U4.1 (VIN)
- net at R3.2: now also J2.1 (Pin_1)
- net at R4.2: now also J2.3 (Pin_3)
- net MCU_EM4WU6: now reaches U7.13 (PC4)
- net MCU_EM4WU6: now also C32.1, D15.1 (A1), R26.1, R31.1
- net LED1: now reaches U7.53 (PF4)
- net LED1: now also R52.1
- net LED2: now reaches U7.54 (PF5)
- net LED2: now also R53.1
- net MCU_EM4WU5: now reaches U7.62 (PE13)
- net MCU_EM4WU5: now also C25.1, D11.1 (A1), R22.1, R27.1
- new net: J6.1 (Pin_1), R20.2
- new net: J6.2 (Pin_2), R21.1
- new net: J6.3 (Pin_3), R22.2
- new net: D16.2 (A), R52.2
- new net: D17.2 (A), R53.2
Other:
- note added: "SIG1"
- note added: "SIG2"
- note added: "Service"
- note added: "Test LEDs"
- note added: "USER LED"
- note added: "WKUP"
- note removed: "Pulse"
- moved on the sheet: C1, C10, C11, C12, C13, C14, C15, C16, C17, C18, C19, C2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
