File: Hardware/GSMLinkModem/GSMLinkModem.sch (KiCad schematic (older format))
At the start: 170 parts, among them J1 KLS1-207-1-04-S, J2 KLS1-207-1-04-S, J3 KLS1-207-1-05-S, J4 KLS2-308V-2.54-02P-4S, J5 SIM8051-6-0-14-00-A, J6 KLS2-308V-2.54-03P-4S, J7 KLS1-207-1-04-S, J8 KLS1-207-1-02-S, J9 1909763-1, Q1 BC847C, Q2 AO3419, Q3 BC847C, Q4 BC847C, Q5 BC847C, Q6 AO3419, Q7 BC847C, SW1 SKQGAKE010, U1 BC66NADA-04-STD, U2 TXS0108EPW, U3 TPS63900, U4 ISL21080DIH310Z-TK, U5 AT25SF321B-SSHB-T, U6 MIC5504-3.3YM5, U7 EFM32TG11B320F128GQ64-B, U8 LIS3DH, U9 Si7055-A20, Y1 32.768kHz, Y2 DNP

Commit message: new: Work in progress
Parts:
- removed C18, C19: 10nF, Capacitor_SMD:C_0805_2012Metric_Pad1.18x1.45mm_HandSolder, symbol Device:C
- removed J9: 1909763-1, digikey-footprints:UMCoax_Pin_1909763-1, symbol Connector:Conn_Coaxial
- added C14, C16: 10uF, Capacitor_SMD:C_0805_2012Metric, symbol Device:C
- added D14: LED_RED, LED_SMD:LED_0603_1608Metric, symbol Device:LED
- added J?: 1909763-1, digikey-footprints:UMCoax_Pin_1909763-1, symbol dk_Coaxial-Connectors-RF:1909763-1
- C1, C2, C22, C24, C28, C3, C31, C35, C37, C4, C45, C49, C50, C56, C57, C59, C60, C61, C62, C63: footprint Capacitor_SMD:C_0805_2012Metric_Pad1.18x1.45mm_HandSolder -> Capacitor_SMD:C_0402_1005Metric; Description 0.1µF ±10% 25V Ceramic Capacitor X7R 0805 (2012 Metric) -> 0.1µF ±10% 16V Ceramic Capacitor X7R 0402 (1005 Metric); PartNumber CC0805KRX7R8BB104 -> CC0402KRX7R7BB104
- C10, C11, C12, C15, C30, C33, C38, C40, C42, C47, C5, C6, C7, C8, C9: footprint Capacitor_SMD:C_0805_2012Metric_Pad1.18x1.45mm_HandSolder -> Capacitor_SMD:C_0402_1005Metric; Description 18pF ±5% 50V Ceramic Capacitor C0G, NP0 0805 (2012 Metric) -> 18pF ±5% 50V Ceramic Capacitor C0G, NP0 0402 (1005 Metric); PartNumber CC0805JRNPO9BN180 -> CC0402JRNPO9BN180
- C13: renamed from C14; footprint Capacitor_SMD:C_0805_2012Metric_Pad1.18x1.45mm_HandSolder -> Capacitor_SMD:C_0402_1005Metric; Description 18pF ±5% 50V Ceramic Capacitor C0G, NP0 0805 (2012 Metric) -> 18pF ±5% 50V Ceramic Capacitor C0G, NP0 0402 (1005 Metric); PartNumber CC0805JRNPO9BN180 -> CC0402JRNPO9BN180
- C17: value 10nF -> 0.1uF; footprint Capacitor_SMD:C_0805_2012Metric_Pad1.18x1.45mm_HandSolder -> Capacitor_SMD:C_0402_1005Metric; Description 10000pF ±5% 100V Ceramic Capacitor C0G, NP0 1206 (3216 Metr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 -> 0.1µF ±10% 16V Ceramic Capacitor X7R 0402 (1005 Metric); PartNumber CC1206JKNPO0BN103 -> CC0402KRX7R7BB104; Voltage 100V -> 25V
- C18: renamed from C13; footprint Capacitor_SMD:C_1206_3216Metric_Pad1.42x1.75mm_HandSolder -> Capacitor_SMD:C_0805_2012Metric; Description 10µF ±10% 25V Ceramic Capacitor X7R 1206 (3216 Metric) -> 10µF ±20% 16V Ceramic Capacitor X7R 0805 (2012 Metric); PartNumber CC1206KKX7R8BB106 -> CC0805MKX7R7BB106
- C19: renamed from C16; footprint Capacitor_SMD:C_1206_3216Metric_Pad1.42x1.75mm_HandSolder -> Capacitor_SMD:C_0805_2012Metric; Description 10µF ±10% 25V Ceramic Capacitor X7R 1206 (3216 Metric) -> 10µF ±20% 16V Ceramic Capacitor X7R 0805 (2012 Metric); PartNumber CC1206KKX7R8BB106 -> CC0805MKX7R7BB106
- C21, C48, C52: footprint Capacitor_SMD:C_0805_2012Metric_Pad1.18x1.45mm_HandSolder -> Capacitor_SMD:C_0603_1608Metric; Description 1µF ±10% 25V Ceramic Capacitor X7R 0805 (2012 Metric) -> 1µF ±10% 16V Ceramic Capacitor X7R 0603 (1608 Metric); PartNumber CC0805KKX7R8BB105 -> CC0603KRX7R7BB105
- C23, C26, C29, C39, C41, C43, C44, C53, C54, C55, C58: footprint Capacitor_SMD:C_1206_3216Metric_Pad1.42x1.75mm_HandSolder -> Capacitor_SMD:C_0805_2012Metric; Description 10µF ±10% 25V Ceramic Capacitor X7R 1206 (3216 Metric) -> 10µF ±20% 16V Ceramic Capacitor X7R 0805 (2012 Metric); PartNumber CC1206KKX7R8BB106 -> CC0805MKX7R7BB106
- C25, C27, C32: value 10nF -> 18pF; footprint Capacitor_SMD:C_0805_2012Metric_Pad1.18x1.45mm_HandSolder -> Capacitor_SMD:C_0402_1005Metric; Description 10000pF ±5% 100V Ceramic Capacitor C0G, NP0 1206 (3216 Metr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 -> 18pF ±5% 50V Ceramic Capacitor C0G, NP0 0402 (1005 Metric); PartNumber CC1206JKNPO0BN103 -> CC0402JRNPO9BN180; Voltage 100V -> 50V
- C34, C36: footprint Capacitor_SMD:C_0402_1005Metric_Pad0.74x0.62mm_HandSolder -> Capacitor_SMD:C_0402_1005Metric
- C51: footprint Capacitor_SMD:C_0805_2012Metric_Pad1.18x1.45mm_HandSolder -> Capacitor_SMD:C_0805_2012Metric
- D10, D11, D12, D13, D2, D3, D4, D5, D6, D7, D8, D9: value PESD5V0L1UA,115 -> PESD5V0L1UB,115; footprint Diode_SMD:D_SOD-323_HandSoldering -> Diode_SMD:D_SOD-523; Description 5V 3.5A (8/20µs) Ipp ESD protection TVS Diode Surface Mount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 -> 12V Clamp 3.5A (8/20µs) Ipp Tvs Diode Surface Mount SOD-523; PartNumber PESD5V0L1UA,115 -> PESD5V0L1UB,115
- D15: renamed from D14; value PESD5V0L1UA,115 -> PESD5V0L1UB,115; footprint Diode_SMD:D_SOD-323_HandSoldering -> Diode_SMD:D_SOD-523; Description 5V 3.5A (8/20µs) Ipp ESD protection TVS Diode Surface Mount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 -> 12V Clamp 3.5A (8/20µs) Ipp Tvs Diode Surface Mount SOD-523; PartNumber PESD5V0L1UA,115 -> PESD5V0L1UB,115
- D16: renamed from D15; value PESD5V0L1UA,115 -> PESD5V0L1UB,115; footprint Diode_SMD:D_SOD-323_HandSoldering -> Diode_SMD:D_SOD-523; Description 5V 3.5A (8/20µs) Ipp ESD protection TVS Diode Surface Mount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 -> 12V Clamp 3.5A (8/20µs) Ipp Tvs Diode Surface Mount SOD-523; PartNumber PESD5V0L1UA,115 -> PESD5V0L1UB,115
- D17: renamed from D16; footprint LED_SMD:LED_0805_2012Metric_Pad1.15x1.40mm_HandSolder -> LED_SMD:LED_0603_1608Metric; Description Red 640nm LED Indication - Discrete 1.85V 0805 (2012 Metric) -> Red 630nm LED Indication - Discrete 1.95V 0603 (1608 Metric); PartNumber APT2012SRCPRV -> APT1608SURCK
- D18: renamed from D17; footprint LED_SMD:LED_0805_2012Metric_Pad1.15x1.40mm_HandSolder -> LED_SMD:LED_0603_1608Metric; Description Green 570nm LED Indication - Discrete 2.1V 0805 (2012 Metri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 -> Green 570nm LED Indication - Discrete 2.1V 0603 (1608 Metri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; PartNumber APT2012CGCK -> APT1608CGCK
- F1: footprint Fuse:Fuse_1206_3216Metric_Pad1.42x1.75mm_HandSolder -> Fuse:Fuse_1206_3216Metric
- FB1: footprint Inductor_SMD:L_0805_2012Metric_Pad1.15x1.40mm_HandSolder -> Inductor_SMD:L_0402_1005Metric; Description 1 kOhms @ 100MHz 1 Power Line Ferrite Bead 0805 (2012 Metri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 -> 1 kOhms @ 100MHz 1 Ferrite Bead 0402 (1005 Metric) 300mA 65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; PartNumber MPZ2012S102JTD25 -> BLM15AG102SN1D
- Q1, Q3, Q4, Q5, Q7: value BC847C -> BC847CW,115; footprint Package_TO_SOT_SMD:SOT-23 -> Package_TO_SOT_SMD:SOT-323_SC-70; Description Bipolar (BJT) Transistor NPN 45V 100mA 100MHz 250mW Surface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 -> Bipolar (BJT) Transistor NPN 45V 100mA 100MHz 200mW Surface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; PartNumber BC847C,215 -> BC847CW,115
- R1, R12, R13, R14, R2, R20, R22, R23, R24, R26, R3, R4, R44, R46, R47, R48, R49, R5, R6, R7: footprint Resistor_SMD:R_0805_2012Metric_Pad1.15x1.40mm_HandSolder -> Resistor_SMD:R_0402_1005Metric; Description 22 Ohms ±5% 0.125W, 1/8W Chip Resistor 0805 (2012 Metric) T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 -> 22 Ohms ±5% 0.125W, 1/8W Chip Resistor 0402 (1005 Metric) T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; PartNumber RC0805JR-0722RL -> RC0402JR-0722RL
- R10, R17, R21, R25, R28, R43, R52, R53, R8: footprint Resistor_SMD:R_0805_2012Metric_Pad1.15x1.40mm_HandSolder -> Resistor_SMD:R_0402_1005Metric; Description 470 Ohms ±5% 0.125W, 1/8W Chip Resistor 0805 (2012 Metric) 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 -> 470 Ohms ±5% 0.125W, 1/8W Chip Resistor 0402 (1005 Metric) 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; PartNumber RC0805JR-07470RL -> RC0402FR-07470RL
- R11, R15, R16, R18, R19, R27, R29, R30, R31, R33, R35, R37, R40, R45, R51, R9: footprint Resistor_SMD:R_0805_2012Metric_Pad1.15x1.40mm_HandSolder -> Resistor_SMD:R_0402_1005Metric; Description 10 kOhms ±1% 0.125W, 1/8W Chip Resistor 0805 (2012 Metric) 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 -> 10 kOhms ±1% 0.063W, 1/16W Chip Resistor 0402 (1005 Metric)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; PartNumber RC0805FR-0710KP -> RC0402FR-0710KL
- R32: footprint Resistor_SMD:R_0402_1005Metric_Pad0.72x0.64mm_HandSolder -> Resistor_SMD:R_0402_1005Metric
- R34: value 10K -> 470R; footprint Resistor_SMD:R_0805_2012Metric_Pad1.15x1.40mm_HandSolder -> Resistor_SMD:R_0402_1005Metric; Description 10 kOhms ±1% 0.125W, 1/8W Chip Resistor 0805 (2012 Metric) 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 -> 470 Ohms ±5% 0.125W, 1/8W Chip Resistor 0402 (1005 Metric) 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; PartNumber RC0805FR-0710KP -> RC0402FR-07470RL
- R36: footprint Resistor_SMD:R_0805_2012Metric_Pad1.15x1.40mm_HandSolder -> Resistor_SMD:R_0402_1005Metric; Description 16.2 kOhms ±1% 0.125W, 1/8W Chip Resistor 0805 (2012 Metric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 -> 16.2 kOhms ±1% 0.063W, 1/16W Chip Resistor 0402 (1005 Metri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; PartNumber RC0805FR-0716K2L -> RC0402FR-0716K2L
- R38: footprint Resistor_SMD:R_0805_2012Metric_Pad1.15x1.40mm_HandSolder -> Resistor_SMD:R_0402_1005Metric; Description 8.25 kOhms ±1% 0.125W, 1/8W Chip Resistor 0805 (2012 Metric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 -> 8.25 kOhms ±1% 0.125W, 1/8W Chip Resistor 0402 (1005 Metric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; PartNumber RC0805FR-078K25L -> RC0402FR-078K25L
- R39: footprint Resistor_SMD:R_0805_2012Metric_Pad1.15x1.40mm_HandSolder -> Resistor_SMD:R_0402_1005Metric; Description 5.11 kOhms ±1% 0.125W, 1/8W Chip Resistor 0805 (2012 Metric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 -> 5.11 kOhms ±1% 0.125W, 1/8W Chip Resistor 0402 (1005 Metric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; PartNumber RC0805FR-075K11L -> RC0402FR-075K11L
- R41: footprint Resistor_SMD:R_0805_2012Metric_Pad1.15x1.40mm_HandSolder -> Resistor_SMD:R_0402_1005Metric; Description 3 MOhms ±1% 0.125W, 1/8W Chip Resistor 0805 (2012 Metric) T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 -> 3 MOhms ±1% 0.125W, 1/8W Chip Resistor 0402 (1005 Metric) T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; PartNumber RC0805FR-073ML -> RC0402FR-073ML
- R42: footprint Resistor_SMD:R_0805_2012Metric_Pad1.15x1.40mm_HandSolder -> Resistor_SMD:R_0402_1005Metric; Description 1 MOhms ±1% 0.125W, 1/8W Chip Resistor 0805 (2012 Metric) T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 -> 1 MOhms ±1% 0.125W, 1/8W Chip Resistor 0402 (1005 Metric) T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; PartNumber RC0805FR-071ML -> RC0402FR-071ML
- R50: footprint Resistor_SMD:R_0805_2012Metric_Pad1.15x1.40mm_HandSolder -> Resistor_SMD:R_0402_1005Metric; PartNumber RC0805JR-072KL -> RC0402FR-072KL
- R54, R55: footprint Resistor_SMD:R_0805_2012Metric_Pad1.15x1.40mm_HandSolder -> Resistor_SMD:R_0402_1005Metric; PartNumber RC0805JR-074K7L -> RC0402JR-074K7L
- U4: footprint Package_TO_SOT_SMD:SOT-23_Handsoldering -> Package_TO_SOT_SMD:SOT-23W
Connections:
- net BC66_ON_OFF: now also U7.33 (PD5); no longer U7.34 (PD6)
- net BC66_PWR: now also U7.32 (PD4); no longer U7.33 (PD5)
- net BC66_RST: now also U7.31 (PD3); no longer U7.32 (PD4)
- net GND: now also C14.2, C16.2, J?.1
- net at C18.1, C19.1, D9.1 (A1)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: now also C14.1, C16.1
- net at C36.1, R32.1: now also J?.2
- removed net NET_STATUS: Q5.3 (C), R34.2, U7.31 (PD3)
- new net: D14.2 (A), R34.2
- new net: D14.1 (K), Q5.3 (C)
Other:
- moved on the sheet: C18, C19

Commit message: new: Work in progress
Parts:
- removed C18, C19, C53: 10uF, Capacitor_SMD:C_0805_2012Metric, symbol Device:C
- removed C51: 10nF, Capacitor_SMD:C_0805_2012Metric, symbol Device:C
- removed R50: 2K, Resistor_SMD:R_0402_1005Metric, symbol Device:R
- removed U4: ISL21080DIH310Z-TK, Package_TO_SOT_SMD:SOT-23W, symbol mylib-symbols:ISL21080DIH310Z-TK
- added H1, H2: MountingHole, MountingHole:MountingHole_3.2mm_M3, symbol Mechanical:MountingHole
- gave numbers to parts that had none: 1
- renumbered C20 to C18, C21 to C19, C22 to C20, C23 to C21, C24 to C22, C25 to C23, C26 to C24, C27 to C25, C28 to C26, C29 to C27, C30 to C28, C31 to C29, C32 to C30, C33 to C31, C34 to C32, C35 to C33, C36 to C34, C37 to C35, C38 to C36, C39 to C37, C40 to C38, C42 to C39, C43 to C40, C44 to C41, C46 to C42, C47 to C43, C41 to C44, C48 to C45, C45 to C46, C49 to C47, C50 to C48, C52 to C49, C54 to C50, C55 to C51, C56 to C52, C57 to C53, C58 to C54, C59 to C55, C60 to C56, C61 to C57, C62 to C58, C63 to C59, R51 to R50, R52 to R51, R53 to R52, R54 to R53, R55 to R54, U5 to U4, U6 to U5, U7 to U6, U8 to U7, U9 to U8
Connections:
- net 3V3_ENBL: now also U6.35 (PD7); no longer U6.17 (PA12)
- net SCL: now also R53.1
- net SDA: no longer R53.1
- net SW_ENBL: now also U6.36 (PD8); no longer U6.6 (PA5)
- net VDDA: now also C44.1, C46.1, FB1.2
- net V_SELECT: now also U6.34 (PD6); no longer U6.18 (PA13)
Other:
- note added: "FLASH"
- note added: "Filter to reduce noise at AVDD pin (bead + 1x10uF+1x0.1uF)"
- note added: "Mounting"
- note removed: "FLASH SPI"
- note removed: "Filter to reduce noise at AVDD pin (1x10uF+2x0.1uF) + 1.024V micropower referece"
- moved on the sheet: C44, C46, C47, C51, C52, C53, C56, C57, FB1, R45, TP1, TP2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

Commit message: new: Work in progress
Parts:
- removed R44: 22R, Resistor_SMD:R_0402_1005Metric, symbol Device:R
- removed SW1: SKQGAKE010, Button_Switch_SMD:SW_SPST_SKQG_WithStem, symbol Switch:SW_Push
- C54: value 10uF -> 1uF; footprint Capacitor_SMD:C_0805_2012Metric -> Capacitor_SMD:C_0603_1608Metric; Description 10µF ±20% 16V Ceramic Capacitor X7R 0805 (2012 Metric) -> 1µF ±10% 16V Ceramic Capacitor X7R 0603 (1608 Metric); PartNumber CC0805MKX7R7BB106 -> CC0603KRX7R7BB105
- renumbered C47 to C46, C46 to C47, R45 to R44, R46 to R45, R47 to R46, R48 to R47, R49 to R48, R50 to R49, R51 to R50, R52 to R51, R53 to R52, R54 to R53
Connections:
- net +3V3: now also C54.1; no longer C54.2
- net GND: now also C54.2; no longer C54.1
- net MCU_RESET: now also C46.1, R44.2, U6.20 (~RESET~)
