File: Hardware/GSMLinkModem/GSMLinkModem.sch (KiCad schematic (older format))
At the start: 165 parts, among them J1 KLS1-207-1-04-S, J2 KLS1-207-1-04-S, J3 KLS1-207-1-05-S, J4 KLS2-308V-2.54-02P-4S, J5 SIM8051-6-0-14-00-A, J6 KLS2-308V-2.54-03P-4S, J7 KLS1-207-1-04-S, J8 KLS1-207-1-02-S, J9 1909763-1, Q1 BC847CW,115, Q2 AO3419, Q3 BC847CW,115, Q4 BC847CW,115, Q5 BC847CW,115, Q6 AO3419, Q7 BC847CW,115, U1 BC66NADA-04-STD, U2 TXS0108EPW, U3 TPS63900, U4 AT25SF321B-SSHB-T, U5 MIC5504-3.3YM5, U6 EFM32TG11B320F128GQ64-B, U7 LIS3DH, U8 Si7055-A20, Y1 32.768kHz, Y2 DNP

Commit message: new: Work in progress
Parts:
- removed C18: 820uF, Capacitor_THT:CP_Radial_D8.0mm_P3.50mm, symbol Device:CP1
- removed R44: 10K, Resistor_SMD:R_0402_1005Metric, symbol Device:R
- added C?: 11mF, mylib-footprints:CAPCP3225X100N, symbol Device:CP1
- added R?: 470R, Resistor_SMD:R_0402_1005Metric, symbol Device:R
- added R?: 22R, Resistor_SMD:R_0402_1005Metric, symbol Device:R
- C36, C38: value 18pF -> DNP
Connections:
- net 3V3_ENBL: now also U6.18 (PA13); no longer U6.35 (PD7)
- net GND: now also C?.2
- net SCL: no longer R53.1
- net SDA: now also R53.1
- net SW_ENBL: now also U6.19 (PA14); no longer U6.36 (PD8)
- net V_SELECT: now also U6.17 (PA12); no longer U6.34 (PD6)
- net at C41.1, R41.2, R42.1: now also R?.2; no longer U6.11 (PB5)
- new net: C?.1, R?.1
- new net: R?.2, U6.36 (PD8)
- new net VBAT_MON: R?.1, U6.35 (PD7)
Other:
- note added: "RTC EDLC"
- moved on the sheet: C41, R41, R42

Commit message: new: Work in progress
Parts:
- gave numbers to parts that had none: 3
- renumbered C19 to C18, C20 to C19, C21 to C20, C22 to C21, C23 to C22, C24 to C23, C25 to C24, C26 to C25, C27 to C26, C28 to C27, C29 to C28, C30 to C29, C31 to C30, C32 to C31, C33 to C32, C34 to C33, C35 to C34, C36 to C35, C41 to C36, C42 to C41, C43 to C42, C44 to C43, C45 to C44, C46 to C45, C47 to C46, C48 to C47, C49 to C48, C50 to C49, C51 to C50, C52 to C51, C53 to C52, C54 to C53, C55 to C54, C56 to C55, C57 to C56, R41 to R36, R42 to R37, R36 to R38, R37 to R39, R38 to R40, R39 to R42, R40 to R43, R43 to R44, R52 to R53, R53 to R54

Commit message: new: Work in progress
Connections:
- net CS: now also U6.47 (PC14); no longer U6.43 (PE6)
- net SDO: now also U6.48 (PC15); no longer U6.57 (PE8)
Changed lines of the file:
@@
 Wire Wire Line
 	16800 11500 17500 11500
-Wire Wire Line
-	16800 11700 17650 11700
-Text GLabel 17650 11700 2    50   Input ~ 0
+Text GLabel 14400 13100 0    50   Input ~ 0
 CS
 Text GLabel 17650 11800 2    50   Input ~ 0
@@
 	1    0    0    -1
 $EndComp
-Text GLabel 17650 11900 2    50   Input ~ 0
+Text GLabel 14400 13200 0    50   Input ~ 0
 SDO
-Wire Wire Line
-	17650 11900 16800 11900
 Wire Notes Line
 	17450 11200 17450 12000
@@
 Text Notes 18900 10950 2    50   ~ 0
 RTC EDLC
+Wire Wire Line
+	14800 13100 14400 13100
+Wire Wire Line
+	14800 13200 14400 13200
 $EndSCHEMATC

Commit message: new: Work in progress
Other:
- note added: "LIS3DHTR ADR/CS pins"
- note removed: "RESET button"
Changed lines of the file:
@@
 Wire Notes Line
 	14350 12400 13650 12400
-Text Notes 13850 12700 0    50   ~ 0
+Text Notes 14350 12400 0    50   ~ 0
 Service
 Text GLabel 10550 7400 2    50   Input ~ 0
@@
 Wire Notes Line
 	14400 10350 14400 11050
-Text Notes 14150 14050 1    50   ~ 0
-RESET button
 Wire Wire Line
 	14250 14050 14250 13950
@@
 Wire Wire Line
 	14800 13200 14400 13200
+Wire Notes Line
+	14150 13000 14150 13300
+Wire Notes Line
+	14150 13300 14450 13300
+Wire Notes Line
+	14450 13300 14450 13000
+Wire Notes Line
+	14450 13000 14150 13000
+Text Notes 13700 12800 0    50   ~ 0
+LIS3DHTR ADR/CS pins
+Wire Notes Line
+	14300 13000 14300 12800
 $EndSCHEMATC

Commit message: new: Rev. 1.0
Parts:
- removed TP1: VBAT_line, TestPoint:TestPoint_THTPad_D1.5mm_Drill0.7mm, symbol Connector:TestPoint
- removed TP2: 3V3_line, TestPoint:TestPoint_THTPad_D1.5mm_Drill0.7mm, symbol Connector:TestPoint
- removed TP3: VCC_line, TestPoint:TestPoint_THTPad_D1.5mm_Drill0.7mm, symbol Connector:TestPoint
- removed TP4: GND, TestPoint:TestPoint_THTPad_D1.5mm_Drill0.7mm, symbol Connector:TestPoint
- C31, C33: DoNotPlaceStatus (none) -> DNP
- C35, C38, C39, C42: value DNP -> 18pF; DoNotPlaceStatus (none) -> DNP
- Y2: value DNP -> ABM8-48-000MHZ; DoNotPlaceStatus (none) -> DNP
Other:
- note removed: "Test points"
- moved on the sheet: H1, H2
