File: Hardware/GSMLinkModem/GSMLinkModem.kicad_pcb (KiCad board)
At the start: 2 copper layers, 104 x 54.5 mm, 170 parts, among them J1 KLS1-207-1-04-S, J2 KLS1-207-1-04-S, J3 KLS1-207-1-05-S, J4 KLS2-308V-2.54-02P-4S, J5 SIM8051-6-0-14-00-A, J6 KLS2-308V-2.54-03P-4S, J7 KLS1-207-1-04-S, J8 KLS1-207-1-02-S, J9 1909763-1, Q1 BC847C, Q2 AO3419, Q3 BC847C, Q4 BC847C, Q5 BC847C, Q6 AO3419, Q7 BC847C, SW1 SKQGAKE010, U1 BC66NADA-04-STD, U2 TXS0108EPW, U3 TPS63900, U4 ISL21080DIH310Z-TK, U5 AT25SF321B-SSHB-T, U6 MIC5504-3.3YM5, U7 EFM32TG11B320F128GQ64-B, U8 LIS3DH, U9 Si7055-A20, Y1 32.768kHz, Y2 DNP

Commit message: new: Work in progress
Parts:
- removed the C18 at (158.3, 40.8)
- removed the C44 at (102.1, 68.5)
- removed C62, C63: 0.1uF, Capacitor_SMD:C_0805_2012Metric_Pad1.18x1.45mm_HandSolder
- added C20: 0.1uF, Capacitor_SMD:C_0402_1005Metric, F.Cu at (148.0, 90.8)
- added C46: 1uF, Capacitor_SMD:C_0603_1608Metric, F.Cu at (170.4, 101.0)
- added D18: LED_GREEN, LED_SMD:LED_0603_1608Metric, F.Cu at (155.0, 64.7)
- C1, C10, C11, C12, C15, C2, C22, C3, C30, C35, C38, C4, C5, C57, C59, C6, C60, C61, C7, C8, C9: footprint Capacitor_SMD:C_0805_2012Metric_Pad1.18x1.45mm_HandSolder -> Capacitor_SMD:C_0402_1005Metric
- C13, C23: value 10uF -> 18pF; footprint Capacitor_SMD:C_1206_3216Metric_Pad1.42x1.75mm_HandSolder -> Capacitor_SMD:C_0402_1005Metric
- C14: value 18pF -> 10uF; footprint Capacitor_SMD:C_0805_2012Metric_Pad1.18x1.45mm_HandSolder -> Capacitor_SMD:C_0805_2012Metric
- C16, C39, C41, C53: footprint Capacitor_SMD:C_1206_3216Metric_Pad1.42x1.75mm_HandSolder -> Capacitor_SMD:C_0805_2012Metric
- C17: value 10nF -> 0.1uF; footprint Capacitor_SMD:C_0805_2012Metric_Pad1.18x1.45mm_HandSolder -> Capacitor_SMD:C_0402_1005Metric
- C19: value 10nF -> 1uF; footprint Capacitor_SMD:C_0805_2012Metric_Pad1.18x1.45mm_HandSolder -> Capacitor_SMD:C_0603_1608Metric
- C21, C52: value 1uF -> 10uF; footprint Capacitor_SMD:C_0805_2012Metric_Pad1.18x1.45mm_HandSolder -> Capacitor_SMD:C_0805_2012Metric
- C24, C37, C56: value 0.1uF -> 10uF; footprint Capacitor_SMD:C_0805_2012Metric_Pad1.18x1.45mm_HandSolder -> Capacitor_SMD:C_0805_2012Metric
- C25: value 10nF -> 18pF; footprint Capacitor_SMD:C_0805_2012Metric_Pad1.18x1.45mm_HandSolder -> Capacitor_SMD:C_0402_1005Metric
- C26, C29, C43, C54, C55, C58: value 10uF -> 0.1uF; footprint Capacitor_SMD:C_1206_3216Metric_Pad1.42x1.75mm_HandSolder -> Capacitor_SMD:C_0402_1005Metric
- C27, C51: value 10nF -> 10uF; footprint Capacitor_SMD:C_0805_2012Metric_Pad1.18x1.45mm_HandSolder -> Capacitor_SMD:C_0805_2012Metric
- C28, C31: value 0.1uF -> 18pF; footprint Capacitor_SMD:C_0805_2012Metric_Pad1.18x1.45mm_HandSolder -> Capacitor_SMD:C_0402_1005Metric
- C32: value 10nF -> DNP; footprint Capacitor_SMD:C_0805_2012Metric_Pad1.18x1.45mm_HandSolder -> Capacitor_SMD:C_0402_1005Metric
- C33: value 18pF -> 0.1uF; footprint Capacitor_SMD:C_0805_2012Metric_Pad1.18x1.45mm_HandSolder -> Capacitor_SMD:C_0402_1005Metric
- C34: footprint Capacitor_SMD:C_0402_1005Metric_Pad0.74x0.62mm_HandSolder -> Capacitor_SMD:C_0402_1005Metric
- C36: value DNP -> 18pF; footprint Capacitor_SMD:C_0402_1005Metric_Pad0.74x0.62mm_HandSolder -> Capacitor_SMD:C_0402_1005Metric
- C40: value 18pF -> DNP; footprint Capacitor_SMD:C_0805_2012Metric_Pad1.18x1.45mm_HandSolder -> Capacitor_SMD:C_0402_1005Metric
- C42: value DNP -> 10uF; footprint Capacitor_SMD:C_0805_2012Metric_Pad1.18x1.45mm_HandSolder -> Capacitor_SMD:C_0805_2012Metric
- C45: value 0.1uF -> DNP; footprint Capacitor_SMD:C_0805_2012Metric_Pad1.18x1.45mm_HandSolder -> Capacitor_SMD:C_0402_1005Metric
- C47: value DNP -> 0.1uF; footprint Capacitor_SMD:C_0805_2012Metric_Pad1.18x1.45mm_HandSolder -> Capacitor_SMD:C_0402_1005Metric
- C48: value 1uF -> 0.1uF; footprint Capacitor_SMD:C_0805_2012Metric_Pad1.18x1.45mm_HandSolder -> Capacitor_SMD:C_0402_1005Metric
- C49: value 0.1uF -> 10nF; footprint Capacitor_SMD:C_0805_2012Metric_Pad1.18x1.45mm_HandSolder -> Capacitor_SMD:C_0805_2012Metric
- C50: value 0.1uF -> 1uF; footprint Capacitor_SMD:C_0805_2012Metric_Pad1.18x1.45mm_HandSolder -> Capacitor_SMD:C_0603_1608Metric
- D10, D11, D12, D13, D15, D2, D3, D4, D5, D6, D7, D8, D9: value PESD5V0L1UA,115 -> PESD5V0L1UB,115; footprint Diode_SMD:D_SOD-323_HandSoldering -> Diode_SMD:D_SOD-523
- D14: value PESD5V0L1UA,115 -> LED_RED; footprint Diode_SMD:D_SOD-323_HandSoldering -> LED_SMD:LED_0603_1608Metric
- D16: value LED_RED -> PESD5V0L1UB,115; footprint LED_SMD:LED_0805_2012Metric_Pad1.15x1.40mm_HandSolder -> Diode_SMD:D_SOD-523
- D17: value LED_GREEN -> LED_RED; footprint LED_SMD:LED_0805_2012Metric_Pad1.15x1.40mm_HandSolder -> LED_SMD:LED_0603_1608Metric
- F1: footprint Fuse:Fuse_1206_3216Metric_Pad1.42x1.75mm_HandSolder -> Fuse:Fuse_1206_3216Metric
- FB1: footprint Inductor_SMD:L_0805_2012Metric_Pad1.15x1.40mm_HandSolder -> Inductor_SMD:L_0402_1005Metric
- Q1, Q3, Q4, Q5, Q7: value BC847C -> BC847CW,115; footprint Package_TO_SOT_SMD:SOT-23 -> Package_TO_SOT_SMD:SOT-323_SC-70
- R1, R10, R11, R12, R13, R14, R15, R16, R17, R18, R19, R2, R20, R21, R22, R23, R24, R25, R26, R27, R28, R29, R3, R30, R31, R33, R35, R36, R37, R38, R39, R4, R40, R41, R42, R43, R44, R45, R46, R47, R48, R49, R5, R50, R51, R52, R53, R54, R55, R6, R7, R8, R9: footprint Resistor_SMD:R_0805_2012Metric_Pad1.15x1.40mm_HandSolder -> Resistor_SMD:R_0402_1005Metric
- R32: footprint Resistor_SMD:R_0402_1005Metric_Pad0.72x0.64mm_HandSolder -> Resistor_SMD:R_0402_1005Metric
- R34: value 10K -> 470R; footprint Resistor_SMD:R_0805_2012Metric_Pad1.15x1.40mm_HandSolder -> Resistor_SMD:R_0402_1005Metric
- U4: footprint Package_TO_SOT_SMD:SOT-23_Handsoldering -> Package_TO_SOT_SMD:SOT-23W
- moved TP1 110.9 mm to (173.7, 85.5)
- moved TP2 110.9 mm to (176.4, 85.5)
- moved TP3 110.9 mm to (170.9, 85.5)
- moved TP4 110.9 mm to (179.2, 85.5)
- moved U2 107.3 mm to (194.4, 128.1)
- moved J9 101.1 mm to (202.2, 106.6), turned to 270 degrees
- moved R32 100.6 mm to (198.8, 106.6), turned to 180 degrees
- moved C34 97.5 mm to (199.3, 105.0), turned to 90 degrees
- moved U7 97.1 mm to (153.7, 109.9)
- moved C17 96.4 mm to (192.2, 144.2), turned to 90 degrees
- moved R28 95.9 mm to (188.6, 127.5)
- moved C15 94.9 mm to (178.0, 125.8), turned to 270 degrees
- moved R18 89.7 mm to (187.8, 144.1), turned to 270 degrees
- moved C24 89.5 mm to (199.3, 117.7), turned to 90 degrees
- moved C19 89.4 mm to (180.8, 143.7)
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- renumbered C20 to C18, C46 to C44
Connections:
- C13 pad 1: Net-(C13-Pad1) -> MCU_SWCLK
- C14 pad 1: MCU_SWCLK -> Net-(C14-Pad1)
- C16 pad 1: Net-(C13-Pad1) -> Net-(C14-Pad1)
- C19 pad 1: Net-(C13-Pad1) -> SIM_VDD
- C21 pad 1: SIM_VDD -> +BATT
- C22 pad 1: +BATT -> VBUS
- C23 pad 1: +BATT -> MCU_EM4WU5
- C24 pad 1: VBUS -> +1V8
- C25 pad 1: MCU_EM4WU5 -> MCU_EM4WU4
- C26 pad 1: +1V8 -> +BATT
- C27 pad 1: MCU_EM4WU4 -> +BATT
- C28 pad 1: +BATT -> EXT_TXD_DBG
- C29 pad 1: +BATT -> +3V3
- C30 pad 1: EXT_TXD_DBG -> MCU_EM4WU6
- C31 pad 1: +3V3 -> EXT_RXD_DBG
- C32 pad 1: MCU_EM4WU6 -> Net-(C32-Pad1)
- C33 pad 1: EXT_RXD_DBG -> +1V8
- C35 pad 1: +1V8 -> +3V3
- C37 pad 1: +3V3 -> VCC
- C39 pad 1: VCC -> Net-(C39-Pad1)
- C41 pad 1: Net-(C41-Pad1) -> VCC
- C43 pad 1: VCC -> Net-(C39-Pad1)
- C45 pad 1: Net-(C41-Pad1) -> Net-(C45-Pad1)
- C48 pad 1: VCC -> Net-(C48-Pad1)
- C49 pad 1: Net-(C49-Pad1) -> VDDA
- C51 pad 1: VDDA -> Net-(C51-Pad1)
- C52 pad 1: Net-(C52-Pad1) -> +3V3
- C53 pad 1: Net-(C53-Pad1) -> +BATT
- C54 pad 1: +3V3 -> +BATT
- C56 pad 1: +BATT -> GND
- C56 pad 2: GND -> +3V3
- C57 pad 1: +BATT -> GND
- C57 pad 2: GND -> +3V3
- C58 pad 1: GND -> +BATT
- C58 pad 2: +3V3 -> GND
- C59 pad 1: GND -> +BATT
- C59 pad 2: +3V3 -> GND
- C60 pad 1: +BATT -> +3V3
- C61 pad 1: +BATT -> +3V3
- D14 pad 1: EXT_RXD_DBG -> Net-(D14-Pad1)
- D14 pad 2: GND -> Net-(D14-Pad2)
- D15 pad 1: MCU_EM4WU6 -> EXT_RXD_DBG
- D16 pad 1: GND -> MCU_EM4WU6
- D16 pad 2: Net-(D16-Pad2) -> GND
- D9 pad 1: Net-(C13-Pad1) -> Net-(C14-Pad1)
- FB1 pad 2: Net-(C41-Pad1) -> Net-(C39-Pad1)
- J9 pad 1: Net-(C36-Pad1) -> GND
- J9 pad 2: GND -> Net-(C34-Pad1)
- Q2 pad 3: Net-(C13-Pad1) -> Net-(C14-Pad1)
- Q5 pad 3: NET_STATUS -> Net-(D14-Pad1)
- Q6 pad 3: Net-(C50-Pad1) -> Net-(C48-Pad1)
- R32 pad 1: Net-(C36-Pad1) -> Net-(C34-Pad1)
- R32 pad 2: Net-(C34-Pad1) -> Net-(C32-Pad1)
- R34 pad 2: NET_STATUS -> Net-(D14-Pad2)
- R41 pad 2: Net-(C44-Pad1) -> Net-(C42-Pad1)
- R42 pad 1: Net-(C44-Pad1) -> Net-(C42-Pad1)
- R44 pad 1: Net-(C49-Pad1) -> Net-(C47-Pad1)
- R45 pad 2: Net-(C49-Pad1) -> Net-(C47-Pad1)
- R50 pad 2: Net-(C53-Pad1) -> Net-(C51-Pad1)
- R52 pad 2: Net-(D16-Pad2) -> Net-(D17-Pad2)
- R53 pad 2: Net-(D17-Pad2) -> Net-(D18-Pad2)
- U1 pad 35: Net-(C34-Pad1) -> Net-(C32-Pad1)
- U1 pad 42: Net-(C13-Pad1) -> Net-(C14-Pad1)
- U1 pad 43: Net-(C13-Pad1) -> Net-(C14-Pad1)
- U4 pad 1: Net-(C41-Pad1) -> Net-(C39-Pad1)
- U5 pad 8: Net-(C50-Pad1) -> Net-(C48-Pad1)
- U7 pad 11: Net-(C44-Pad1) -> Net-(C42-Pad1)
- U7 pad 15: Net-(C38-Pad1) -> Net-(C36-Pad1)
- U7 pad 16: Net-(C40-Pad1) -> Net-(C38-Pad1)
- U7 pad 20: Net-(C49-Pad1) -> Net-(C47-Pad1)
- U7 pad 24: Net-(C42-Pad1) -> Net-(C40-Pad1)
- U7 pad 25: Net-(C47-Pad1) -> Net-(C45-Pad1)
- U7 pad 31: NET_STATUS -> BC66_RST
- U7 pad 32: BC66_RST -> BC66_PWR
- U7 pad 33: BC66_PWR -> BC66_ON_OFF
- U7 pad 34: BC66_ON_OFF -> Net-(U7-Pad34)
- U7 pad 40: Net-(C52-Pad1) -> Net-(C50-Pad1)
- Y1 pad 1: Net-(C38-Pad1) -> Net-(C36-Pad1)
- Y1 pad 2: Net-(C40-Pad1) -> Net-(C38-Pad1)
- Y2 pad 1: Net-(C42-Pad1) -> Net-(C40-Pad1)
- Y2 pad 3: Net-(C47-Pad1) -> Net-(C45-Pad1)
Routing:
- net GND: track 15.5 -> 88.6 mm, vias 13 -> 65
- net Net-(C15-Pad1): track 0.00 -> 40.9 mm, vias 0 -> 3
- net BC66_TXD_AUX: track 0.00 -> 26.5 mm
- net +1V8: track 0.00 -> 26.5 mm, vias 0 -> 2
- net BC66_RXD_AUX: track 0.00 -> 24.6 mm
- net SIM_VDD: track 0.00 -> 23.3 mm
- net Net-(C10-Pad1): track 0.00 -> 23.0 mm, vias 0 -> 3
- net Net-(C12-Pad1): track 0.00 -> 16.6 mm, vias 0 -> 3
- net Net-(C17-Pad1): track 0.00 -> 15.3 mm
- net +BATT: track 8.29 -> 22.8 mm
- net BC66_TXD: track 0.00 -> 8.03 mm
- net +3V3: track 0.00 -> 8.00 mm, vias 0 -> 2
- net SIM_DATA: track 0.00 -> 7.86 mm
- net BC66_RXD: track 0.00 -> 6.84 mm
- net BC66_RESET: track 0.00 -> 6.50 mm
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- added copper zone on F.Cu, net +BATT
- added copper zone on F.Cu, net Net-(C14-Pad1)
- added copper zone on F.Cu, net VCC
Other:
- outline, holes or cut-outs redrawn
- copper layers 2 -> 4

Commit message: new: Work in progress
Parts:
- removed C60, C61: 0.1uF, Capacitor_SMD:C_0402_1005Metric
- removed R55: 4.7K, Resistor_SMD:R_0402_1005Metric
- removed U9: Si7055-A20, Package_DFN_QFN:DFN-6-1EP_3x3mm_P1mm_EP1.5x2.4mm
- added H1: MountingHole, MountingHole:MountingHole_3.2mm_M3, F.Cu at (199.5, 135.0)
- added H2: MountingHole, MountingHole:MountingHole_3.2mm_M3, F.Cu at (104.5, 107.0)
- C39: value 10uF -> DNP; footprint Capacitor_SMD:C_0805_2012Metric -> Capacitor_SMD:C_0402_1005Metric
- C40: value DNP -> 10uF; footprint Capacitor_SMD:C_0402_1005Metric -> Capacitor_SMD:C_0805_2012Metric
- C42: value 10uF -> 820uF; footprint Capacitor_SMD:C_0805_2012Metric -> Capacitor_THT:CP_Radial_D8.0mm_P3.50mm
- C43: value 0.1uF -> DNP
- C44: value 820uF -> 10uF; footprint Capacitor_THT:CP_Radial_D8.0mm_P3.50mm -> Capacitor_SMD:C_0805_2012Metric
- C45: value DNP -> 1uF; footprint Capacitor_SMD:C_0402_1005Metric -> Capacitor_SMD:C_0603_1608Metric
- C46: value 1uF -> 0.1uF; footprint Capacitor_SMD:C_0603_1608Metric -> Capacitor_SMD:C_0402_1005Metric
- C49: value 10nF -> 1uF; footprint Capacitor_SMD:C_0805_2012Metric -> Capacitor_SMD:C_0603_1608Metric
- C50: value 1uF -> 10uF; footprint Capacitor_SMD:C_0603_1608Metric -> Capacitor_SMD:C_0805_2012Metric
- C52, C53, C56: value 10uF -> 0.1uF; footprint Capacitor_SMD:C_0805_2012Metric -> Capacitor_SMD:C_0402_1005Metric
- C54: value 0.1uF -> 10uF; footprint Capacitor_SMD:C_0402_1005Metric -> Capacitor_SMD:C_0805_2012Metric
- R50: value 2K -> 10K
- R51: value 10K -> 470R
- R53: value 470R -> 4.7K
- U4: value ISL21080DIH310Z-TK -> AT25SF321B-SSHB-T; footprint Package_TO_SOT_SMD:SOT-23W -> Package_SO:SOIC-8_3.9x4.9mm_P1.27mm
- U5: value AT25SF321B-SSHB-T -> MIC5504-3.3YM5; footprint Package_SO:SOIC-8_3.9x4.9mm_P1.27mm -> Package_TO_SOT_SMD:SOT-23-5
- U6: value MIC5504-3.3YM5 -> EFM32TG11B320F128GQ64-B; footprint Package_TO_SOT_SMD:SOT-23-5 -> Package_QFP:TQFP-64_10x10mm_P0.5mm
- U7: value EFM32TG11B320F128GQ64-B -> LIS3DH; footprint Package_QFP:TQFP-64_10x10mm_P0.5mm -> Package_LGA:LGA-16_3x3mm_P0.5mm_LayoutBorder3x5y
- U8: value LIS3DH -> Si7055-A20; footprint Package_LGA:LGA-16_3x3mm_P0.5mm_LayoutBorder3x5y -> Package_DFN_QFN:DFN-6-1EP_3x3mm_P1mm_EP1.5x2.4mm
- moved C54 97.2 mm to (142.6, 162.6), turned to 90 degrees
- moved C55 92.7 mm to (148.2, 165.0)
- moved C30 84.6 mm to (165.8, 38.3)
- moved C23 84.6 mm to (162.7, 40.4)
- moved SW1 84.6 mm to (148.9, 40.7)
- moved C59 84.6 mm to (138.7, 150.8), turned to 90 degrees
- moved Q5 84.5 mm to (194.4, 137.7), turned to 90 degrees
- moved C58 81.5 mm to (137.4, 162.8)
- moved R30 80.9 mm to (193.6, 140.5), turned to 270 degrees
- moved C22 69.5 mm to (170.3, 137.9)
- moved C6 69.5 mm to (169.8, 141.8)
- moved R10 64.4 mm to (185.7, 129.3), turned to 270 degrees
- moved Y2 60.4 mm to (142.3, 114.1), turned to 270 degrees
- moved R15 60.2 mm to (184.6, 129.3), turned to 90 degrees
- moved R51 58.2 mm to (131.6, 142.2)
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Connections:
- C40 pad 1: Net-(C40-Pad1) -> VCC
- C41 pad 1: VCC -> Net-(C41-Pad1)
- C42 pad 1: Net-(C42-Pad1) -> VCC
- C43 pad 1: Net-(C39-Pad1) -> Net-(C43-Pad1)
- C44 pad 1: VCC -> VDDA
- C45 pad 1: Net-(C45-Pad1) -> VCC
- C46 pad 1: VCC -> VDDA
- C49 pad 1: VDDA -> Net-(C49-Pad1)
- C50 pad 1: Net-(C50-Pad1) -> +3V3
- C51 pad 1: Net-(C51-Pad1) -> +BATT
- C52 pad 1: +3V3 -> +BATT
- C54 pad 1: +BATT -> GND
- C54 pad 2: GND -> +3V3
- C55 pad 1: +BATT -> GND
- C55 pad 2: GND -> +3V3
- C56 pad 1: GND -> +BATT
- C56 pad 2: +3V3 -> GND
- C57 pad 1: GND -> +BATT
- C57 pad 2: +3V3 -> GND
- C58 pad 1: +BATT -> +3V3
- C59 pad 1: +BATT -> +3V3
- FB1 pad 2: Net-(C39-Pad1) -> VDDA
- R41 pad 2: Net-(C42-Pad1) -> Net-(C41-Pad1)
- R42 pad 1: Net-(C42-Pad1) -> Net-(C41-Pad1)
- R50 pad 1: VDDA -> 3V3_ENBL
- R50 pad 2: Net-(C51-Pad1) -> GND
- R51 pad 1: 3V3_ENBL -> LED1
- R51 pad 2: GND -> Net-(D17-Pad2)
- R52 pad 1: LED1 -> LED2
- R52 pad 2: Net-(D17-Pad2) -> Net-(D18-Pad2)
- R53 pad 1: LED2 -> SCL
- R53 pad 2: Net-(D18-Pad2) -> +3V3
- R54 pad 1: SDA -> SCL
- U4 pad 1: Net-(C39-Pad1) -> MCU_CS
- U4 pad 2: VDDA -> MCU_MISO
- U4 pad 3: GND -> Net-(U4-Pad3)
- U5 pad 1: MCU_CS -> VCC
- U5 pad 2: MCU_MISO -> GND
- U5 pad 3: Net-(U5-Pad3) -> 3V3_ENBL
- U5 pad 4: GND -> Net-(U5-Pad4)
- U5 pad 5: MCU_MOSI -> +3V3
- U6 pad 1: VCC -> Net-(R46-Pad1)
- U6 pad 2: GND -> Net-(R47-Pad1)
- U6 pad 3: 3V3_ENBL -> Net-(R48-Pad1)
- U6 pad 4: Net-(U6-Pad4) -> Net-(R49-Pad1)
- U6 pad 5: +3V3 -> FLASH_PWR
- U7 pad 1: Net-(R46-Pad1) -> +3V3
- U7 pad 10: Net-(U7-Pad10) -> GND
- U7 pad 11: Net-(C42-Pad1) -> INT1
- U7 pad 12: Net-(U7-Pad12) -> GND
- U7 pad 13: MCU_EM4WU6 -> Net-(U7-Pad13)
- U7 pad 14: Net-(U7-Pad14) -> +3V3
- U7 pad 15: Net-(C36-Pad1) -> Net-(U7-Pad15)
- U7 pad 16: Net-(C38-Pad1) -> Net-(U7-Pad16)
- U7 pad 2: Net-(R47-Pad1) -> Net-(U7-Pad2)
- U7 pad 3: Net-(R48-Pad1) -> Net-(U7-Pad3)
- U7 pad 4: Net-(R49-Pad1) -> SCL
- U7 pad 5: FLASH_PWR -> GND
- U7 pad 6: SW_ENBL -> SDA
- U7 pad 7: +BATT -> SDO
- U7 pad 8: GND -> CS
- U8 pad 1: +3V3 -> SDA
- U8 pad 2: Net-(U8-Pad2) -> GND
- U8 pad 4: SCL -> Net-(U8-Pad4)
- U8 pad 5: GND -> +3V3
- U8 pad 6: SDA -> SCL
- U8 pad 7: SDO -> (no net)
- Y2 pad 1: Net-(C40-Pad1) -> Net-(C39-Pad1)
- Y2 pad 3: Net-(C45-Pad1) -> Net-(C43-Pad1)
Routing:
- net VBUS: track 5.59 -> 118.6 mm
- net +3V3: track 8.00 -> 82.3 mm, vias 2 -> 4
- net GND: track 88.6 -> 133.0 mm, vias 65 -> 88
- net MCU_TX1: track 0.00 -> 44.0 mm, vias 0 -> 1
- net MCU_RI: track 0.00 -> 43.3 mm, vias 0 -> 1
- net MCU_RX1: track 0.00 -> 43.1 mm, vias 0 -> 1
- net EXT_TXD: track 0.00 -> 38.5 mm, vias 0 -> 1
- net EXT_RXD: track 0.00 -> 38.2 mm, vias 0 -> 1
- net EXT_TXD_DBG: track 0.00 -> 37.7 mm, vias 0 -> 1
- net EXT_RXD_DBG: track 0.00 -> 36.6 mm, vias 0 -> 1
- net BC66_TXD_DBG: track 0.00 -> 31.9 mm, vias 0 -> 2
- net BC66_RXD_DBG: track 0.00 -> 31.3 mm, vias 0 -> 2
- net SIM_VDD: track 23.3 -> 54.3 mm, vias 0 -> 5
- net BC66_RST: track 0.00 -> 23.2 mm, vias 0 -> 1
- net BC66_PWR: track 0.00 -> 22.0 mm
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- added copper zone on In2.Cu, net +BATT
- added copper zone on In1.Cu, net GND
- added copper zone on In2.Cu, net VCC

Commit message: new: Work in progress
Parts:
- removed the R44 at (137.8, 75.7)
- removed the R53 at (149.4, 67.8)
- removed SW1: SKQGAKE010, Button_Switch_SMD:SW_SPST_SKQG_WithStem
- added R52: 4.7K, Resistor_SMD:R_0402_1005Metric, F.Cu at (149.4, 67.8)
- C54: value 10uF -> 1uF; footprint Capacitor_SMD:C_0805_2012Metric -> Capacitor_SMD:C_0603_1608Metric
- moved C54 77.1 mm to (158.7, 87.2), turned to 0 degrees
- moved R20 74.7 mm to (114.6, 116.2), turned to 90 degrees
- moved D5 73.6 mm to (121.9, 113.7)
- moved C28 70.5 mm to (131.2, 115.4), turned to 270 degrees
- moved U8 64.7 mm to (121.7, 128.6)
- moved R40 64.2 mm to (169.2, 145.4), turned to 90 degrees
- moved C2 62.2 mm to (118.6, 115.4), turned to 90 degrees
- moved D12 61.1 mm to (129.8, 113.6), turned to 180 degrees
- moved Q7 60.7 mm to (166.9, 145.3), turned to 180 degrees
- moved R24 59.0 mm to (130.2, 115.4), turned to 270 degrees
- moved R50 57.6 mm to (127.2, 84.8), turned to 180 degrees
- moved R14 57.2 mm to (120.8, 98.8), turned to 90 degrees
- moved R12 56.4 mm to (125.2, 98.8), turned to 90 degrees
- moved Q6 56.4 mm to (166.9, 142.1), turned to 90 degrees
- moved C6 55.9 mm to (120.6, 115.4), turned to 270 degrees
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- renumbered C47 to C46, C46 to C47, R45 to R44, R46 to R45, R47 to R46, R48 to R47, R49 to R48, R50 to R49, R51 to R50, R52 to R51, R54 to R53
Connections:
- C46 pad 1: Net-(C47-Pad1) -> MCU_RESET
- C54 pad 1: GND -> +3V3
- C54 pad 2: +3V3 -> GND
- R44 pad 2: Net-(C47-Pad1) -> MCU_RESET
- U6 pad 20: Net-(C47-Pad1) -> MCU_RESET
Routing:
- net 3V3_ENBL: track 4.64 -> 30.4 mm
- net GND: track 133.0 -> 157.0 mm, vias 88 -> 110
- net +3V3: track 82.3 -> 106.0 mm
- net MCU_TX0: track 0.00 -> 21.3 mm
- net Net-(J6-Pad3): track 0.00 -> 20.3 mm
- net MCU_RX0: track 0.00 -> 20.0 mm
- net Net-(J6-Pad2): track 0.00 -> 17.7 mm
- net Net-(J6-Pad1): track 0.00 -> 14.5 mm
- net MCU_RESET: track 0.00 -> 12.2 mm
- net Net-(J8-Pad1): track 0.00 -> 10.4 mm
- net VBUS: track 118.6 -> 128.4 mm
- net MCU_SWDIO: track 0.00 -> 9.25 mm
- net Net-(J8-Pad2): track 0.00 -> 7.37 mm
- net MCU_SWCLK: track 0.00 -> 6.84 mm
- net +BATT: track 41.7 -> 48.1 mm, vias 21 -> 20
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
Commit message: new: Work in progress
Parts:
- removed the C18 at (158.3, 98.0)
- removed the R44 at (147.1, 69.8)
- added C57: 11mF, mylib-footprints:CAPCP3225X100N, F.Cu at (159.6, 108.0)
- added R41: 22R, Resistor_SMD:R_0402_1005Metric, F.Cu at (154.9, 107.7)
- added R52: 470R, Resistor_SMD:R_0402_1005Metric, F.Cu at (159.7, 105.3)
- C35: renamed from C36; value 18pF -> DNP
- C38: value 18pF -> DNP
- moved R25 104.0 mm to (105.9, 133.1), turned to 180 degrees
- moved C29 99.0 mm to (110.2, 120.2), turned to 270 degrees
- moved C22 93.4 mm to (114.2, 120.2), turned to 270 degrees
- moved R22 86.0 mm to (113.2, 120.2), turned to 270 degrees
- moved D16 85.7 mm to (109.4, 117.6), turned to 90 degrees
- moved R21 82.8 mm to (105.9, 136.0), turned to 180 degrees
- moved C25 81.0 mm to (105.9, 132.1)
- moved D13 80.3 mm to (111.7, 117.6), turned to 90 degrees
- moved C19 72.2 mm to (105.9, 135.0)
- moved D11 67.8 mm to (114.0, 117.6), turned to 90 degrees
- moved TP1 64.9 mm to (110.5, 85.5)
- moved TP2 64.9 mm to (113.3, 85.5)
- moved TP3 64.9 mm to (107.8, 85.5)
- moved TP4 64.9 mm to (116.0, 85.5)
- moved C34 56.6 mm to (168.3, 115.8), turned to 270 degrees
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- renumbered C19 to C18, C20 to C19, C21 to C20, C22 to C21, C23 to C22, C24 to C23, C25 to C24, C26 to C25, C27 to C26, C28 to C27, C29 to C28, C30 to C29, C31 to C30, C32 to C31, C33 to C32, C34 to C33, C35 to C34, C41 to C36, C42 to C41, C43 to C42, C44 to C43, C45 to C44, C46 to C45, C47 to C46, C48 to C47, C49 to C48, C50 to C49, C51 to C50, C52 to C51, C53 to C52, C54 to C53, C55 to C54, C56 to C55, C57 to C56, R41 to R36, R42 to R37, R36 to R38, R37 to R39, R38 to R40, R39 to R42, R40 to R43, R43 to R44, R52 to R53, R53 to R54
Connections:
- C36 pad 1: Net-(C41-Pad1) -> Net-(C36-Pad1)
- R36 pad 2: Net-(C41-Pad1) -> Net-(C36-Pad1)
- R37 pad 1: Net-(C41-Pad1) -> Net-(C36-Pad1)
- R54 pad 1: SCL -> SDA
- U6 pad 11: Net-(C41-Pad1) -> Net-(U6-Pad11)
- U6 pad 17: Net-(U6-Pad17) -> V_SELECT
- U6 pad 18: Net-(U6-Pad18) -> 3V3_ENBL
- U6 pad 19: Net-(U6-Pad19) -> SW_ENBL
- U6 pad 34: V_SELECT -> Net-(U6-Pad34)
- U6 pad 35: 3V3_ENBL -> VBAT_MON
- U6 pad 36: SW_ENBL -> Net-(R52-Pad2)
Routing:
- net EXT_TXD: track 40.9 -> 107.3 mm, vias 1 -> 2
- net EXT_RXD: track 40.6 -> 105.4 mm, vias 1 -> 2
- net V_SELECT: track 4.16 -> 32.7 mm, vias 0 -> 2
- net MCU_RESET: track 12.2 -> 38.6 mm, vias 0 -> 2
- net MCU_RI: track 43.3 -> 68.4 mm, vias 1 -> 2
- net MCU_TX0: track 21.3 -> 43.7 mm
- net MCU_RX0: track 20.0 -> 41.4 mm
- net Net-(J6-Pad3): track 20.3 -> 0.00 mm
- net BC66_PWR: track 22.0 -> 3.86 mm, vias 0 -> 1
- net Net-(J6-Pad1): track 14.5 -> 0.33 mm
- net SCL: track 0.00 -> 13.0 mm
- net Net-(J6-Pad2): track 17.7 -> 4.98 mm
- net 3V3_ENBL: track 30.4 -> 42.0 mm, vias 1 -> 2
- net Net-(C47-Pad1): track 0.00 -> 8.56 mm
- net MCU_SWDIO: track 9.25 -> 17.1 mm
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
Commit message: new: Work in progress
Parts:
- moved C53 1.36 mm to (156.8, 96.0), turned to 270 degrees
- moved C54 1.30 mm to (155.1, 95.2), turned to 180 degrees
- moved U7 0.81 mm to (154.1, 97.5)
- moved R29 0.11 mm to (150.3, 96.3)
- moved C34 0.10 mm to (168.4, 115.8)
- moved R50 0.10 mm to (149.2, 96.3)
Routing:
- net +3V3: track 111.3 -> 148.6 mm, vias 6 -> 10
- net Net-(J6-Pad3): track 0.00 -> 19.4 mm
- net GND: track 162.0 -> 180.1 mm, vias 116 -> 127
- net Net-(J6-Pad1): track 0.33 -> 14.3 mm
- net Net-(J8-Pad2): track 0.00 -> 5.91 mm
- net MCU_EM4WU4: track 0.00 -> 5.79 mm
- net SDO: track 0.00 -> 3.49 mm
- net CS: track 5.53 -> 2.43 mm
- net LED1: track 0.00 -> 2.91 mm
- net MCU_RESET: track 38.6 -> 41.3 mm
- net LED2: track 0.00 -> 2.71 mm
- net MCU_EM4WU6: track 0.00 -> 2.56 mm
- net MCU_EM4WU5: track 0.00 -> 2.54 mm
- net INT1: track 4.20 -> 1.81 mm
- net SW_ENBL: track 3.45 -> 5.70 mm, vias 0 -> 1
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- added copper zone on F.Cu, net GND

Commit message: new: Work in progress
Parts:
- moved D18 20.8 mm to (132.8, 102.8)
- moved D17 20.7 mm to (131.0, 102.8)
- moved C50 20.4 mm to (149.6, 116.9), turned to 0 degrees
- moved TP4 6.15 mm to (122.2, 85.5)
- moved C59 4.98 mm to (141.0, 98.0)
- moved U8 1.61 mm to (138.2, 97.2), turned to 0 degrees
- moved C58 0.70 mm to (156.4, 101.7)
- moved R53 0.70 mm to (157.4, 101.7)
- moved R54 0.70 mm to (155.4, 101.7)
- moved C12 0.40 mm to (180.3, 125.8)
- moved R6 0.40 mm to (180.3, 123.2)
- moved D1 0.40 mm to (183.4, 125.9)
- moved R31 0.39 mm to (137.8, 107.2)
- moved TP3 0.30 mm to (107.5, 85.5)
- moved C10 0.30 mm to (179.2, 125.8)
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Connections:
- U6 pad 43: CS -> Net-(U6-Pad43)
- U6 pad 47: Net-(U6-Pad47) -> CS
- U6 pad 48: Net-(U6-Pad48) -> SDO
- U6 pad 57: SDO -> Net-(U6-Pad57)
Routing:
- net EXT_TXD_DBG: track 41.2 -> 150.3 mm
- net Net-(Q7-Pad1): track 1.32 -> 80.5 mm, vias 0 -> 2
- net MCU_EM4WU4: track 5.79 -> 61.8 mm, vias 0 -> 2
- net MCU_EM4WU6: track 2.56 -> 53.2 mm, vias 0 -> 2
- net MCU_EM4WU5: track 2.54 -> 52.7 mm, vias 0 -> 2
- net EXT_RXD_DBG: track 40.2 -> 85.9 mm
- net GND: track 180.1 -> 217.2 mm, vias 127 -> 143
- net MCU_SWCLK: track 12.3 -> 46.1 mm, vias 0 -> 2
- net SDA: track 7.38 -> 39.7 mm, vias 0 -> 2
- net BC66_RST: track 24.1 -> 55.1 mm
- net Net-(R47-Pad1): track 0.00 -> 29.7 mm, vias 0 -> 2
- net SW_ENBL: track 5.70 -> 34.1 mm, vias 1 -> 2
- net Net-(R45-Pad1): track 0.00 -> 27.7 mm, vias 0 -> 2
- net SCL: track 14.6 -> 41.3 mm, vias 0 -> 2
- net MCU_SWDIO: track 17.1 -> 42.8 mm
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Other:
- net class Default: clearance 0.2 -> 0.15
- rule trace_clearance: 0.2 -> 0.15

Commit message: new: Rev. 1.0
Parts:
- removed TP1: VBAT_line, TestPoint:TestPoint_THTPad_D1.5mm_Drill0.7mm
- removed TP2: 3V3_line, TestPoint:TestPoint_THTPad_D1.5mm_Drill0.7mm
- removed TP3: VCC_line, TestPoint:TestPoint_THTPad_D1.5mm_Drill0.7mm
- removed TP4: GND, TestPoint:TestPoint_THTPad_D1.5mm_Drill0.7mm
- C35, C38, C39, C42: value DNP -> 18pF
- Y2: value DNP -> ABM8-48-000MHZ
Routing:
- net EXT_TXD_DBG: track 150.3 -> 108.4 mm
- net +3V3: track 162.2 -> 169.1 mm
- net Net-(C15-Pad1): track 34.8 -> 31.6 mm
- net SIM_VDD: track 54.5 -> 56.6 mm
- net MCU_SWCLK: track 46.1 -> 44.0 mm
- net GND: track 217.2 -> 218.9 mm, vias 143 -> 223
- net BC66_RESET: track 13.0 -> 13.9 mm
- net Net-(C10-Pad1): track 22.6 -> 21.9 mm
- net Net-(J2-Pad1): track 4.25 -> 4.88 mm
- net SDA: track 39.7 -> 39.2 mm
- added copper zone on B.Cu, net GND
Other:
- board text added: "+V"
- board text added: "104.ua NB-IoT"
- board text added: "ANT"
- board text added: "AUX CON"
- board text added: "BAT"
- board text added: "CLK"
- board text added: "DIO"
- board text added: "GND"
- board text added: "LINK AUX"
- board text added: "LINK MAIN"
- board text added: "MCU DEBUG"
- board text added: "MCU UART"
- board text added: "NET LED"
- board text added: "REED"
- board text added: "RX"
- board text added: "SERVICE"
- board text added: "SIG1"
- board text added: "SIG2"
- board text added: "STATUS"
- board text added: "TX"
- board text added: "V+"
- board text added: "rev. 1.0"
- board text added: "~RST~"
