File: Hardware/Smart104.ua_V3.sch (KiCad schematic (older format))
At the start: 162 parts, among them J1 KLS1-207-1-04-S, J2 KLS1-207-1-04-S, J3 KLS1-207-1-05-S, J4 KLS2-308V-2.54-02P-4S, J5 SIM8051-6-0-14-00-A, J6 KLS2-308V-2.54-03P-4S, J7 KLS1-207-1-04-S, J8 KLS1-207-1-02-S, J9 1909763-1, Q1 BC847CW,115, Q2 AO3419, Q3 BC847CW,115, Q4 BC847CW,115, Q5 BC847CW,115, Q6 AO3419, Q7 BC847CW,115, U1 BC66NADA-04-STD, U2 TXS0108EPW, U3 TPS63900, U4 AT25SF321B-SSHB-T, U5 MIC5504-3.3YM5, U6 EFM32TG11B320F128GQ64-B, U7 LIS3DH, U8 Si7055-A20, Y1 32.768kHz, Y2 ABM8-48-000MHZ

Commit message: new: Rev. 1.0 gerbers/fixes_2
Changed lines of the file:
@@
 External connectors
-Wire Notes Line
-	5050 8500 11250 8500
 Wire Notes Line
 	5050 14350 11250 14350
@@
 Wire Wire Line
 	17600 12250 17800 12250
-Text Notes 17500 14200 0    50   ~ 0
+Text Notes 17400 14200 0    50   ~ 0
 Connect reed switch here
 Text Notes 17200 14100 0    50   ~ 0
@@
 	5000 14350 4550 14350
 Wire Notes Line
-	4950 8500 4550 8500
-Wire Notes Line
 	14600 12600 14600 14250
 Wire Notes Line
@@
 	1    0    0    -1
 $EndComp
+Wire Notes Line
+	4550 8500 11250 8500
 $EndSCHEMATC

Commit message: fix: Rev. 1.0 connector added, pcb fixes
Parts:
- added C3, C4, C7, C8: 18pF, Capacitor_SMD:C_0402_1005Metric, symbol Device:C
- added C54: 100uF, Capacitor_Tantalum_SMD:CP_EIA-3216-18_Kemet-A, symbol Device:CP1
- added C55: 1uF, Capacitor_SMD:C_0603_1608Metric, symbol Device:C
- added C66: 10uF, Capacitor_SMD:C_0805_2012Metric, symbol Device:C
- added D1, D3, D4, D5: PESD5V0L1UB,115, Diode_SMD:D_SOD-523, symbol Diode:SM6T7V5A
- added D21: BAT46JFILM, Diode_SMD:D_SOD-323, symbol Device:D_Schottky
- added J1: 5013310707, Connector_Molex:Molex_Pico-Clasp_501331-0707_1x07-1MP_P1.00mm_Vertical, symbol Connector:Conn_01x07_Male
- added R1, R2, R3, R4: 22R, Resistor_SMD:R_0402_1005Metric, symbol Device:R
- added R56: 10K, Resistor_SMD:R_0402_1005Metric, symbol Device:R
- added U8: MCP1727-3302E_MF, Package_DFN_QFN:VDFN-8-1EP_2x2mm_P0.5mm_EP0.9x1.7mm, symbol mylib-symbols:MCP1727-3302E_MF
- C45: renamed from C41; value 820uF -> 1000uF; Description 820µF 6.3V Aluminum - Polymer Capacitors Radial, Can 16mOhm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 -> 1000µF 6.3V Aluminum - Polymer Capacitors Radial, Can 15mOh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; PartNumber A750KK827M0JAAE016 -> A750KK108M0JAAE015
- renumbered C6 to C10, C7 to C11, C8 to C12, C9 to C13, C10 to C14, C11 to C15, C12 to C16, C13 to C17, C14 to C18, C15 to C19, C16 to C20, C17 to C21, C18 to C22, C19 to C23, C20 to C24, C21 to C25, C22 to C26, C23 to C27, C24 to C28, C25 to C29, C26 to C30, C27 to C31, C28 to C32, C29 to C33, C30 to C34, C31 to C35, C32 to C36, C33 to C37, C34 to C38, C35 to C39, C36 to C40, C37 to C41, C38 to C42, C39 to C43, C40 to C44, C42 to C46, C43 to C47, C44 to C48, C45 to C49, C3 to C5, C46 to C50, C47 to C51, C48 to C52, C49 to C53, C50 to C56, C51 to C57, C53 to C58, C54 to C59, C4 to C6, C52 to C60, C55 to C61, C56 to C62, C57 to C63, C58 to C64, C59 to C65, C5 to C9, D6 to D10, D7 to D11, D8 to D12, D9 to D13, D10 to D14, D11 to D15, D12 to D16, D13 to D17, D14 to D18, D15 to D19, D1 to D2, D16 to D20, D17 to D22, D18 to D23, D2 to D6, D3 to D7, D4 to D8, D5 to D9, J9 to J10, J1 to J2, J2 to J3, J3 to J4, J4 to J5, J5 to J6, J6 to J7, J7 to J8, J8 to J9, R6 to R10, R7 to R11, R8 to R12, R9 to R13, R10 to R14, R11 to R15, R12 to R16, R13 to R17, R14 to R18, R15 to R19, R16 to R20, R17 to R21, R18 to R22, R19 to R23, R20 to R24, R21 to R25, R22 to R26, R23 to R27, R24 to R28, R25 to R29, R26 to R30, R27 to R31, R28 to R32, R29 to R33, R30 to R34, R31 to R35, R32 to R36, R33 to R37, R34 to R38, R35 to R39, R36 to R40, R37 to R41, R38 to R42, R39 to R43, R40 to R44, R41 to R45, R42 to R46, R43 to R47, R44 to R48, R45 to R49, R1 to R5, R46 to R50, R47 to R51, R48 to R52, R49 to R53, R50 to R54, R51 to R55, R52 to R57, R53 to R58, R54 to R59, R2 to R6, R3 to R7, R4 to R8, R5 to R9, U8 to U9
Connections:
- net labels added: +3.3VADC, +3.3VP, ADC0, ADC1, GPIO0, GPIO1, SENS_ENBL, VCCQ
- net labels removed: VBUS, VDDA
- wire segments 608 -> 693
Other:
- note added: "1x100uF + 1x10uF bulk decoupling + 100nF per power pin"
- note added: "ADC Inputs\n"
- note added: "ADC inputs"
- note added: "External GPIO"
- note added: "External sensors"
- note added: "External sensors regulator"
- note added: "GPIO output"
- note added: "PB11 - EM4WU7"
- note added: "Power output"
- note removed: "1x10uF bulk decoupling + 100nF per power pin"
- moved on the sheet: C56, C57, C60, C61, C62
