File: Hardware/Smart104.ua_V3_rev2.kicad_pcb (KiCad board)
At the start: 4 copper layers, 104 x 54.5 mm, 181 parts, among them J1 5013310707, J10 1909763-1, J2 KLS1-207-1-04-S, J3 KLS1-207-1-04-S, J4 KLS1-207-1-05-S, J5 KLS2-308V-2.54-02P-4S, J6 SIM8051-6-0-14-00-A, J7 KLS2-308V-2.54-03P-4S, J8 KLS1-207-1-04-S, J9 KLS1-207-1-02-S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

Commit message: new: Rev. 1.0 LGA-16 footprint fixed, minor fixes
Parts:
- U7: footprint Package_LGA:LGA-16_3x3mm_P0.5mm_LayoutBorder3x5y -> mylib-footprints:LGA-16_3x3mm_P0.5mm_fixed
- moved C58 0.50 mm to (157.3, 96.0)
- moved C59 0.30 mm to (155.1, 94.9)
Routing:
- net Net-(L1-Pad1): track 3.56 -> 0.00 mm
- net INT1: track 8.38 -> 10.5 mm
- net +BATT: track 58.5 -> 60.4 mm
- net GND: track 227.1 -> 225.2 mm, vias 243 -> 242
- net MCU_EM4WU4: track 68.1 -> 66.5 mm
- net +3V3: track 151.6 -> 153.1 mm
- net +3.3VP: track 66.3 -> 67.1 mm
Other:
- board text added: "RF ANT"
- board text added: "SERV"
- board text added: "rev. 2.0"
- board text removed: "ANT"
- board text removed: "rev. 1.0"
