File: Hardware/Smart104.ua_V3_rev2.sch (KiCad schematic (older format))
At the start: 181 parts, among them J1 5013310707, J10 1909763-1, J2 KLS1-207-1-04-S, J3 KLS1-207-1-04-S, J4 KLS1-207-1-05-S, J5 KLS2-308V-2.54-02P-4S, J6 SIM8051-6-0-14-00-A, J7 KLS2-308V-2.54-03P-4S, J8 KLS1-207-1-04-S, J9 KLS1-207-1-02-S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

Commit message: new: Rev. 1.0 LGA-16 footprint fixed, minor fixes
Parts:
- U7: footprint Package_LGA:LGA-16_3x3mm_P0.5mm_LayoutBorder3x5y -> mylib-footprints:LGA-16_3x3mm_P0.5mm_fixed
Changed lines of the file:
@@
 F 0 "U7" H 16250 7750 50  0000 C CNN
 F 1 "LIS3DH" H 16300 7650 50  0000 C CNN
-F 2 "Package_LGA:LGA-16_3x3mm_P0.5mm_LayoutBorder3x5y" H 16700 6150 50  0001 C CNN
+F 2 "mylib-footprints:LGA-16_3x3mm_P0.5mm_fixed" H 16700 6150 50  0001 C CNN
 F 3 "https://www.digikey.com/en/products/detail/stmicroelectronics/LIS3DHTR/2334338" H 16400 7100 50  0001 C CNN
 F 4 "Accelerometer X, Y, Z Axis ±2g, 4g, 8g, 16g 0.5Hz ~ 625Hz 16-LGA (3x3)" H 16600 7200 50  0001 C CNN "Description"
@@
 	17650 3300 17650 3550
 $Comp
-L power:VCCQ #PWR?
+L power:VCCQ #PWR0144
 U 1 1 61F87472
 P 18350 2750
-F 0 "#PWR?" H 18350 2600 50  0001 C CNN
+F 0 "#PWR0144" H 18350 2600 50  0001 C CNN
 F 1 "VCCQ" H 18365 2923 50  0000 C CNN
 F 2 "" H 18350 2750 50  0001 C CNN
@@
 $EndComp
 $Comp
-L power:VCCQ #PWR?
+L power:VCCQ #PWR0153
 U 1 1 61F8AF92
 P 4600 2000
-F 0 "#PWR?" H 4600 1850 50  0001 C CNN
+F 0 "#PWR0153" H 4600 1850 50  0001 C CNN
 F 1 "VCCQ" H 4500 2150 50  0000 C CNN
 F 2 "" H 4600 2000 50  0001 C CNN
